File: hardware/bno085-i2c-board/bno085-i2c-board.kicad_sch (KiCad schematic)
At the start: 0 parts

Commit message: started schematic
Parts:
- added C1: C_Polarized, symbol Device:C_Polarized
- added U1: ~, symbol BNO08x:BNO085
Connections:
- new net: C1.1, U1.9 (CAP)
- new net +3.3V: U1.10 (CLKSEL0), U1.28 (VDDIO), U1.3 (VDD)
- new net GND: C1.2, U1.2 (GND), U1.25 (GNDIO), U1.26 (XOUT32/CLKSEL1)
Changed lines of the file:
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@@
 (kicad_sch (version 20230121) (generator eeschema)
   (paper "A4")
+  (junction (at 170.18 114.3) (diameter 0) (color 0 0 0 0)
+  )
+  (junction (at 129.54 114.3) (diameter 0) (color 0 0 0 0)
+  )
+  (wire (pts (xy 167.64 113.03) (xy 170.18 113.03))
+    (stroke (width 0) (type default))
+  )
+  (wire (pts (xy 132.08 115.57) (xy 129.54 115.57))
+    (stroke (width 0) (type default))
+  )
+  (wire (pts (xy 129.54 115.57) (xy 129.54 114.3))
+    (stroke (width 0) (type default))
+  )
+  (wire (pts (xy 170.18 113.03) (xy 170.18 114.3))
+    (stroke (width 0) (type default))
+  )
+  (wire (pts (xy 129.54 113.03) (xy 129.54 114.3))
+    (stroke (width 0) (type default))
+  )
+  (wire (pts (xy 118.11 88.9) (xy 132.08 88.9))
+    (stroke (width 0) (type default))
+  )
+  (wire (pts (xy 132.08 113.03) (xy 129.54 113.03))
+    (stroke (width 0) (type default))
+  )
+  (wire (pts (xy 170.18 115.57) (xy 170.18 114.3))
+    (stroke (width 0) (type default))
+  )
+  (wire (pts (xy 167.64 115.57) (xy 170.18 115.57))
+    (stroke (width 0) (type default))
+  )
+  (symbol (lib_id "Device:C_Polarized") (at 114.3 88.9 270) (unit 1)
+    (in_bom yes) (on_board yes) (dnp no) (fields_autoplaced)
+    (property "Reference" "C1" (at 115.189 81.28 90)
+      (effects (font (size 1.27 1.27)))
+    )
+    (property "Value" "C_Polarized" (at 115.189 83.82 90)
+      (effects (font (size 1.27 1.27)))
+    )
+    (property "Footprint" "" (at 110.49 89.8652 0)
+      (effects (font (size 1.27 1.27)) hide)
+    )
+    (property "Datasheet" "~" (at 114.3 88.9 0)
+      (effects (font (size 1.27 1.27)) hide)
+    )
+    (pin "1")
+    (pin "2")
+    (instances
+      (project "bno085-i2c-board"
+        (path "/a6bdf641-e64e-4bd0-89ab-89241b3a6e60"
+          (reference "C1") (unit 1)
+        )
+      )
+    )
+  )
+  (symbol (lib_id "power:GND") (at 129.54 114.3 270) (unit 1)
+    (in_bom yes) (on_board yes) (dnp no) (fields_autoplaced)
+    (property "Reference" "#PWR02" (at 123.19 114.3 0)
+      (effects (font (size 1.27 1.27)) hide)
+    )
+    (property "Value" "GND" (at 125.73 114.3 90)
+      (effects (font (size 1.27 1.27)) (justify right))
+    )
+    (property "Footprint" "" (at 129.54 114.3 0)
+      (effects (font (size 1.27 1.27)) hide)
+    )
+    (property "Datasheet" "" (at 129.54 114.3 0)
+      (effects (font (size 1.27 1.27)) hide)
+    )
+    (pin "1")
+    (instances
+      (project "bno085-i2c-board"
+        (path "/a6bdf641-e64e-4bd0-89ab-89241b3a6e60"
+          (reference "#PWR02") (unit 1)
+        )
+      )
+    )
+  )
+  (symbol (lib_id "BNO08x:BNO085") (at 149.86 93.98 0) (unit 1)
+    (in_bom yes) (on_board yes) (dnp no) (fields_autoplaced)
+    (property "Reference" "U1" (at 154.3559 67.31 0)
+      (effects (font (size 1.27 1.27)) (justify left))
+    )
+    (property "Value" "~" (at 149.86 93.98 0)
+      (effects (font (size 1.27 1.27)))
+    )
+    (property "Footprint" "" (at 149.86 93.98 0)
+      (effects (font (size 1.27 1.27)) hide)
+    )
+    (property "Datasheet" "" (at 149.86 93.98 0)
+      (effects (font (size 1.27 1.27)) hide)
+    )
+    (pin "1")
+    (pin "10")
+    (pin "11")
+    (pin "12")
+    (pin "13")
+    (pin "14")
+    (pin "15")
+    (pin "16")
+    (pin "17")
+    (pin "18")
+    (pin "19")
+    (pin "2")
+    (pin "20")
+    (pin "21")
+    (pin "22")
+    (pin "23")
+    (pin "24")
+    (pin "25")
+    (pin "26")
+    (pin "27")
+    (pin "28")
+    (pin "3")
+    (pin "4")
+    (pin "5")
+    (pin "6")
+    (pin "7")
+    (pin "8")
+    (pin "9")
+    (instances
+      (project "bno085-i2c-board"
+        (path "/a6bdf641-e64e-4bd0-89ab-89241b3a6e60"
+          (reference "U1") (unit 1)
+        )
+      )
+    )
+  )
+  (symbol (lib_id "power:GND") (at 167.64 88.9 90) (unit 1)
+    (in_bom yes) (on_board yes) (dnp no) (fields_autoplaced)
+    (property "Reference" "#PWR04" (at 173.99 88.9 0)
+      (effects (font (size 1.27 1.27)) hide)
+    )
+    (property "Value" "GND" (at 171.45 88.9 90)
+      (effects (font (size 1.27 1.27)) (justify right))
+    )
+    (property "Footprint" "" (at 167.64 88.9 0)
+      (effects (font (size 1.27 1.27)) hide)
+    )
+    (property "Datasheet" "" (at 167.64 88.9 0)
+      (effects (font (size 1.27 1.27)) hide)
+    )
+    (pin "1")
+    (instances
+      (project "bno085-i2c-board"
+        (path "/a6bdf641-e64e-4bd0-89ab-89241b3a6e60"
+          (reference "#PWR04") (unit 1)
+        )
+      )
+    )
+  )
+  (symbol (lib_id "power:+3.3V") (at 170.18 114.3 270) (unit 1)
+    (in_bom yes) (on_board yes) (dnp no) (fields_autoplaced)
+    (property "Reference" "#PWR01" (at 166.37 114.3 0)
+      (effects (font (size 1.27 1.27)) hide)
+    )
+    (property "Value" "+3.3V" (at 173.99 114.3 90)
+      (effects (font (size 1.27 1.27)) (justify left))
+    )
+    (property "Footprint" "" (at 170.18 114.3 0)
+      (effects (font (size 1.27 1.27)) hide)
+    )
+    (property "Datasheet" "" (at 170.18 114.3 0)
+      (effects (font (size 1.27 1.27)) hide)
+    )
+    (pin "1")
+    (instances
+      (project "bno085-i2c-board"
+        (path "/a6bdf641-e64e-4bd0-89ab-89241b3a6e60"
+          (reference "#PWR01") (unit 1)
+        )
+      )
+    )
+  )
+  (symbol (lib_id "power:+3.3V") (at 132.08 91.44 90) (unit 1)
+    (in_bom yes) (on_board yes) (dnp no) (fields_autoplaced)
+    (property "Reference" "#PWR03" (at 135.89 91.44 0)
+      (effects (font (size 1.27 1.27)) hide)
+    )
+    (property "Value" "+3.3V" (at 128.27 91.44 90)
+      (effects (font (size 1.27 1.27)) (justify left))
+    )
+    (property "Footprint" "" (at 132.08 91.44 0)
+      (effects (font (size 1.27 1.27)) hide)
+    )
+    (property "Datasheet" "" (at 132.08 91.44 0)
+      (effects (font (size 1.27 1.27)) hide)
+    )
+    (pin "1")
+    (instances
+      (project "bno085-i2c-board"
+        (path "/a6bdf641-e64e-4bd0-89ab-89241b3a6e60"
+          (reference "#PWR03") (unit 1)
+        )
+      )
+    )
+  )
+  (symbol (lib_id "power:GND") (at 110.49 88.9 270) (unit 1)
+    (in_bom yes) (on_board yes) (dnp no) (fields_autoplaced)
+    (property "Reference" "#PWR05" (at 104.14 88.9 0)
+      (effects (font (size 1.27 1.27)) hide)
+    )
+    (property "Value" "GND" (at 106.68 88.9 90)
+      (effects (font (size 1.27 1.27)) (justify right))
+    )
+    (property "Footprint" "" (at 110.49 88.9 0)
+      (effects (font (size 1.27 1.27)) hide)
+    )
+    (property "Datasheet" "" (at 110.49 88.9 0)
+      (effects (font (size 1.27 1.27)) hide)
+    )
+    (pin "1")
+    (instances
+      (project "bno085-i2c-board"
+        (path "/a6bdf641-e64e-4bd0-89ab-89241b3a6e60"
+          (reference "#PWR05") (unit 1)
+        )
+      )
+    )
+  )
   (sheet_instances
     (path "/" (page "1"))

Commit message: more schematic
Parts:
- added J1: Conn_01x06_Pin, symbol Connector:Conn_01x06_Pin
- added R1: 10k, symbol Device:R_Small
- added R2, R3, R4, R5: 2.2k, symbol Device:R_Small
Connections:
- net +3.3V: now also R1.2, R2.1, R3.2, R4.1
- net GND: now also U1.17 (SA0/H_MOSI), U1.5 (PS1), U1.6 (PS0/WAKE), J1.5 (Pin_5)
- net at U1.15 (ENV_SCL): now also R2.2
- net at U1.16 (ENV_SDA): now also R3.1
- net at U1.19 (H_SCL/SCK/RX): now also J1.1 (Pin_1), R4.2
- net at U1.20 (H_SDA/H_MISO/TX): now also R5.2
- net at U1.4 (BOOTN): now also R1.1
- new net: J1.2 (Pin_2), R5.1
- no-connect marks 0 -> 2
Other:
- note added: "Assuming no need to update firmware"
- note added: "ENV_SCL & ENV_SDA are pulled high unless we need them for other sensors"
- moved on the sheet: C1

Commit message: schematic
Connections:
- net +3.3V: now also J1.6 (Pin_6)
- net H_SCL: now reaches J1.1 (Pin_1), R4.2, U1.19 (H_SCL/SCK/RX)
- net NRST: now reaches U1.11 (NRST)
- net NRST: now also J1.3 (Pin_3)
- net H_INTN: now reaches U1.14 (H_INTN)
- net H_INTN: now also J1.4 (Pin_4)
- net H_SDA: now reaches J1.2 (Pin_2), R5.1
Other:
- moved on the sheet: J1, R5
Changed lines of the file:
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@@
 (kicad_sch (version 20230121) (generator eeschema)
   (paper "A4")
+  (junction (at 176.53 124.46) (diameter 0) (color 0 0 0 0)
+  )
   (junction (at 170.18 114.3) (diameter 0) (color 0 0 0 0)
   )
@@
   )
   (junction (at 176.53 114.3) (diameter 0) (color 0 0 0 0)
-  )
-  (junction (at 176.53 125.73) (diameter 0) (color 0 0 0 0)
   )
   (junction (at 129.54 114.3) (diameter 0) (color 0 0 0 0)
@@
   (no_connect (at 167.64 86.36))
   (no_connect (at 151.13 123.19))
-  (wire (pts (xy 181.61 104.14) (xy 193.04 104.14))
+  (wire (pts (xy 196.85 111.76) (xy 212.09 111.76))
     (stroke (width 0) (type default))
   )
@@
     (stroke (width 0) (type default))
   )
-  (wire (pts (xy 167.64 104.14) (xy 176.53 104.14))
+  (wire (pts (xy 167.64 104.14) (xy 170.18 104.14))
     (stroke (width 0) (type default))
   )
@@
     (stroke (width 0) (type default))
   )
+  (wire (pts (xy 196.85 114.3) (xy 212.09 114.3))
+    (stroke (width 0) (type default))
+  )
   (wire (pts (xy 146.05 123.19) (xy 146.05 125.73))
     (stroke (width 0) (type default))
@@
     (stroke (width 0) (type default))
   )
+  (wire (pts (xy 176.53 124.46) (xy 187.96 124.46))
+    (stroke (width 0) (type default))
+  )
   (wire (pts (xy 132.08 73.66) (xy 148.59 73.66))
     (stroke (width 0) (type default))
   )
-  (wire (pts (xy 176.53 123.19) (xy 176.53 125.73))
+  (wire (pts (xy 176.53 123.19) (xy 176.53 124.46))
     (stroke (width 0) (type default))
   )
@@
     (stroke (width 0) (type default))
   )
-  (wire (pts (xy 176.53 125.73) (xy 176.53 127))
+  (wire (pts (xy 196.85 109.22) (xy 212.09 109.22))
     (stroke (width 0) (type default))
   )
@@
     (stroke (width 0) (type default))
   )
-  (wire (pts (xy 153.67 123.19) (xy 153.67 127))
+  (wire (pts (xy 153.67 123.19) (xy 153.67 124.46))
     (stroke (width 0) (type default))
   )
@@
     (stroke (width 0) (type default))
   )
+  (wire (pts (xy 119.38 93.98) (xy 132.08 93.98))
+    (stroke (width 0) (type default))
+  )
+  (wire (pts (xy 196.85 106.68) (xy 212.09 106.68))
+    (stroke (width 0) (type default))
+  )
   (wire (pts (xy 129.54 113.03) (xy 129.54 114.3))
     (stroke (width 0) (type default))
@@
     (stroke (width 0) (type default))
   )
+  (wire (pts (xy 175.26 104.14) (xy 180.34 104.14))
+    (stroke (width 0) (type default))
+  )
   (wire (pts (xy 132.08 113.03) (xy 129.54 113.03))
     (stroke (width 0) (type default))
@@
     (stroke (width 0) (type default))
   )
-  (wire (pts (xy 153.67 127) (xy 176.53 127))
+  (wire (pts (xy 153.67 124.46) (xy 176.53 124.46))
     (stroke (width 0) (type default))
   )
@@
     (stroke (width 0) (type default))
   )
-  (wire (pts (xy 193.04 125.73) (xy 193.04 106.68))
-    (stroke (width 0) (type default))
-  )
   (wire (pts (xy 176.53 114.3) (xy 176.53 118.11))
     (stroke (width 0) (type default))
   )
-  (wire (pts (xy 176.53 125.73) (xy 193.04 125.73))
-    (stroke (width 0) (type default))
-  )
   (wire (pts (xy 176.53 114.3) (xy 170.18 114.3))
     (stroke (width 0) (type default))
   )
   (wire (pts (xy 167.64 115.57) (xy 170.18 115.57))
+    (stroke (width 0) (type default))
+  )
+  (wire (pts (xy 119.38 101.6) (xy 132.08 101.6))
     (stroke (width 0) (type default))
   )
@@
   (text "ENV_SCL & ENV_SDA are pulled high \nunless we need them for other sensors"
     (at 73.66 106.68 0)
+    (effects (font (size 1.27 1.27)) (justify left bottom))
+  )
+  (label "H_SDA" (at 196.85 111.76 0) (fields_autoplaced)
+    (effects (font (size 1.27 1.27)) (justify left bottom))
+  )
+  (label "H_INTN" (at 196.85 106.68 0) (fields_autoplaced)
+    (effects (font (size 1.27 1.27)) (justify left bottom))
+  )
+  (label "H_SCL" (at 187.96 124.46 0) (fields_autoplaced)
+    (effects (font (size 1.27 1.27)) (justify left bottom))
+  )
+  (label "H_SDA" (at 180.34 104.14 0) (fields_autoplaced)
+    (effects (font (size 1.27 1.27)) (justify left bottom))
+  )
+  (label "NRST" (at 119.38 93.98 0) (fields_autoplaced)
+    (effects (font (size 1.27 1.27)) (justify left bottom))
+  )
+  (label "H_INTN" (at 119.38 101.6 0) (fields_autoplaced)
+    (effects (font (size 1.27 1.27)) (justify left bottom))
+  )
+  (label "NRST" (at 196.85 109.22 0) (fields_autoplaced)
+    (effects (font (size 1.27 1.27)) (justify left bottom))
+  )
+  (label "H_SCL" (at 196.85 114.3 0) (fields_autoplaced)
     (effects (font (size 1.27 1.27)) (justify left bottom))
   )
@@
     )
   )
-  (symbol (lib_id "Device:R_Small") (at 179.07 104.14 270) (unit 1)
-    (in_bom yes) (on_board yes) (dnp no)
-    (property "Reference" "R5" (at 179.07 109.22 90)
-      (effects (font (size 1.27 1.27)))
-    )
-    (property "Value" "2.2k" (at 179.07 106.68 90)
-      (effects (font (size 1.27 1.27)))
-    )
-    (property "Footprint" "" (at 179.07 104.14 0)
-      (effects (font (size 1.27 1.27)) hide)
-    )
-    (property "Datasheet" "~" (at 179.07 104.14 0)
+  (symbol (lib_id "Device:R_Small") (at 172.72 104.14 270) (unit 1)
+    (in_bom yes) (on_board yes) (dnp no)
+    (property "Reference" "R5" (at 172.72 109.22 90)
+      (effects (font (size 1.27 1.27)))
+    )
+    (property "Value" "2.2k" (at 172.72 106.68 90)
+      (effects (font (size 1.27 1.27)))
+    )
+    (property "Footprint" "" (at 172.72 104.14 0)
+      (effects (font (size 1.27 1.27)) hide)
+    )
+    (property "Datasheet" "~" (at 172.72 104.14 0)
       (effects (font (size 1.27 1.27)) hide)
     )
@@
     )
   )
-  (symbol (lib_id "power:GND") (at 193.04 96.52 270) (unit 1)
-    (in_bom yes) (on_board yes) (dnp no) (fields_autoplaced)
-    (property "Reference" "#PWR010" (at 186.69 96.52 0)
-      (effects (font (size 1.27 1.27)) hide)
-    )
-    (property "Value" "GND" (at 189.23 96.52 90)
+  (symbol (lib_id "power:GND") (at 212.09 104.14 270) (unit 1)
+    (in_bom yes) (on_board yes) (dnp no) (fields_autoplaced)
+    (property "Reference" "#PWR010" (at 205.74 104.14 0)
+      (effects (font (size 1.27 1.27)) hide)
+    )
+    (property "Value" "GND" (at 208.28 104.14 90)
       (effects (font (size 1.27 1.27)) (justify right))
     )
-    (property "Footprint" "" (at 193.04 96.52 0)
-      (effects (font (size 1.27 1.27)) hide)
-    )
-    (property "Datasheet" "" (at 193.04 96.52 0)
+    (property "Footprint" "" (at 212.09 104.14 0)
+      (effects (font (size 1.27 1.27)) hide)
+    )
+    (property "Datasheet" "" (at 212.09 104.14 0)
       (effects (font (size 1.27 1.27)) hide)
     )
@@
   )
   (symbol (lib_id "power:+3.3V") (at 132.08 91.44 90) (unit 1)
-    (in_bom yes) (on_board yes) (dnp no) (fields_autoplaced)
+    (in_bom yes) (on_board yes) (dnp no)
     (property "Reference" "#PWR03" (at 135.89 91.44 0)
       (effects (font (size 1.27 1.27)) hide)
     )
-    (property "Value" "+3.3V" (at 128.27 91.44 90)
+    (property "Value" "+3.3V" (at 129.54 91.44 90)
       (effects (font (size 1.27 1.27)) (justify left))
     )
@@
         (path "/a6bdf641-e64e-4bd0-89ab-89241b3a6e60"
           (reference "#PWR03") (unit 1)
+        )
+      )
+    )
+  )
+  (symbol (lib_id "power:+3.3V") (at 212.09 101.6 90) (unit 1)
+    (in_bom yes) (on_board yes) (dnp no) (fields_autoplaced)
+    (property "Reference" "#PWR012" (at 215.9 101.6 0)
+      (effects (font (size 1.27 1.27)) hide)
+    )
+    (property "Value" "+3.3V" (at 208.28 101.6 90)
+      (effects (font (size 1.27 1.27)) (justify left))
+    )
+    (property "Footprint" "" (at 212.09 101.6 0)
+      (effects (font (size 1.27 1.27)) hide)
+    )
+    (property "Datasheet" "" (at 212.09 101.6 0)
+      (effects (font (size 1.27 1.27)) hide)
+    )
+    (pin "1")
+    (instances
+      (project "bno085-i2c-board"
+        (path "/a6bdf641-e64e-4bd0-89ab-89241b3a6e60"
+          (reference "#PWR012") (unit 1)
         )
       )
@@
     )
   )
-  (symbol (lib_id "Connector:Conn_01x06_Pin") (at 198.12 101.6 180) (unit 1)
-    (in_bom yes) (on_board yes) (dnp no) (fields_autoplaced)
-    (property "Reference" "J1" (at 199.39 99.06 0)
+  (symbol (lib_id "Connector:Conn_01x06_Pin") (at 217.17 109.22 180) (unit 1)
+    (in_bom yes) (on_board yes) (dnp no) (fields_autoplaced)
+    (property "Reference" "J1" (at 218.44 106.68 0)
       (effects (font (size 1.27 1.27)) (justify right))
     )
-    (property "Value" "Conn_01x06_Pin" (at 199.39 101.6 0)
+    (property "Value" "Conn_01x06_Pin" (at 218.44 109.22 0)
       (effects (font (size 1.27 1.27)) (justify right))
     )
-    (property "Footprint" "" (at 198.12 101.6 0)
-      (effects (font (size 1.27 1.27)) hide)
-    )
-    (property "Datasheet" "~" (at 198.12 101.6 0)
-      (effects (font (size 1.27 1.27)) hide)
-    )
+    (property "Footprint" "" (at 217.17 109.22 0)
+      (effects (font (size 1.27 1.27)) hide)
+    )
+    (property "Datasheet" "~" (at 217.17 109.22 0)
+      (effects (font (size 1.27 1.27)) hide)
+    )
