File: hardware/bno085-i2c-board/bno085-i2c-board.kicad_sch (KiCad schematic)
At the start: 8 parts, among them J1 Conn_01x06_Pin

Commit message: pcb
Parts:
- C1: value C_Polarized -> 0.1uF; footprint (none) -> Capacitor_THT:CP_Radial_D5.0mm_P2.00mm
- J1: footprint (none) -> Connector_PinHeader_2.54mm:PinHeader_1x06_P2.54mm_Horizontal
- R1, R2, R3, R4, R5: footprint (none) -> Resistor_SMD:R_01005_0402Metric
- U1: footprint (none) -> Package_LGA:LGA-28_5.2x3.8mm_P0.5mm
Connections:
- net +3.3V: now also J1.2 (Pin_2); no longer J1.6 (Pin_6)
- net GND: now also J1.1 (Pin_1); no longer J1.5 (Pin_5)
- net H_INTN: now also J1.3 (Pin_3); no longer J1.4 (Pin_4)
- net H_SCL: now also J1.5 (Pin_5); no longer J1.1 (Pin_1)
- net H_SDA: now also J1.6 (Pin_6); no longer J1.2 (Pin_2)
- net NRST: now also J1.4 (Pin_4); no longer J1.3 (Pin_3)
Changed lines of the file:
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@@
   (junction (at 132.08 73.66) (diameter 0) (color 0 0 0 0)
   )
-  (junction (at 209.55 101.6) (diameter 0) (color 0 0 0 0)
+  (junction (at 212.09 111.76) (diameter 0) (color 0 0 0 0)
   )
   (junction (at 176.53 114.3) (diameter 0) (color 0 0 0 0)
@@
   (no_connect (at 167.64 86.36))
   (no_connect (at 151.13 123.19))
-  (wire (pts (xy 196.85 111.76) (xy 212.09 111.76))
+  (wire (pts (xy 196.85 101.6) (xy 212.09 101.6))
     (stroke (width 0) (type default))
   )
@@
     (stroke (width 0) (type default))
   )
-  (wire (pts (xy 196.85 114.3) (xy 212.09 114.3))
+  (wire (pts (xy 196.85 104.14) (xy 212.09 104.14))
     (stroke (width 0) (type default))
   )
@@
     (stroke (width 0) (type default))
   )
-  (wire (pts (xy 207.01 101.6) (xy 209.55 101.6))
+  (wire (pts (xy 209.55 111.76) (xy 212.09 111.76))
     (stroke (width 0) (type default))
   )
@@
   )
   (wire (pts (xy 123.19 88.9) (xy 132.08 88.9))
-    (stroke (width 0) (type default))
-  )
-  (wire (pts (xy 209.55 101.6) (xy 212.09 101.6))
     (stroke (width 0) (type default))
   )
@@
     (effects (font (size 1.27 1.27)) (justify left bottom))
   )
-  (label "H_SDA" (at 196.85 111.76 0) (fields_autoplaced)
-    (effects (font (size 1.27 1.27)) (justify left bottom))
-  )
-  (label "H_INTN" (at 196.85 106.68 0) (fields_autoplaced)
+  (label "H_SDA" (at 196.85 101.6 0) (fields_autoplaced)
+    (effects (font (size 1.27 1.27)) (justify left bottom))
+  )
+  (label "NRST" (at 196.85 106.68 0) (fields_autoplaced)
     (effects (font (size 1.27 1.27)) (justify left bottom))
   )
@@
     (effects (font (size 1.27 1.27)) (justify left bottom))
   )
-  (label "NRST" (at 196.85 109.22 0) (fields_autoplaced)
-    (effects (font (size 1.27 1.27)) (justify left bottom))
-  )
-  (label "H_SCL" (at 196.85 114.3 0) (fields_autoplaced)
+  (label "H_INTN" (at 196.85 109.22 0) (fields_autoplaced)
+    (effects (font (size 1.27 1.27)) (justify left bottom))
+  )
+  (label "H_SCL" (at 196.85 104.14 0) (fields_autoplaced)
     (effects (font (size 1.27 1.27)) (justify left bottom))
   )
@@
       (effects (font (size 1.27 1.27)))
     )
-    (property "Value" "C_Polarized" (at 120.269 83.82 90)
-      (effects (font (size 1.27 1.27)))
-    )
-    (property "Footprint" "" (at 115.57 89.8652 0)
+    (property "Value" "0.1uF" (at 120.269 83.82 90)
+      (effects (font (size 1.27 1.27)))
+    )
+    (property "Footprint" "Capacitor_THT:CP_Radial_D5.0mm_P2.00mm" (at 115.57 89.8652 0)
       (effects (font (size 1.27 1.27)) hide)
     )
@@
     )
   )
-  (symbol (lib_id "power:PWR_FLAG") (at 209.55 101.6 0) (unit 1)
-    (in_bom yes) (on_board yes) (dnp no) (fields_autoplaced)
-    (property "Reference" "#FLG01" (at 209.55 99.695 0)
-      (effects (font (size 1.27 1.27)) hide)
-    )
-    (property "Value" "PWR_FLAG" (at 209.55 96.52 0)
-      (effects (font (size 1.27 1.27)))
-    )
-    (property "Footprint" "" (at 209.55 101.6 0)
-      (effects (font (size 1.27 1.27)) hide)
-    )
-    (property "Datasheet" "~" (at 209.55 101.6 0)
+  (symbol (lib_id "power:PWR_FLAG") (at 212.09 111.76 0) (unit 1)
+    (in_bom yes) (on_board yes) (dnp no) (fields_autoplaced)
+    (property "Reference" "#FLG01" (at 212.09 109.855 0)
+      (effects (font (size 1.27 1.27)) hide)
+    )
+    (property "Value" "PWR_FLAG" (at 212.09 106.68 0)
+      (effects (font (size 1.27 1.27)))
+    )
+    (property "Footprint" "" (at 212.09 111.76 0)
+      (effects (font (size 1.27 1.27)) hide)
+    )
+    (property "Datasheet" "~" (at 212.09 111.76 0)
       (effects (font (size 1.27 1.27)) hide)
     )
@@
       (effects (font (size 1.27 1.27)))
     )
-    (property "Footprint" "" (at 158.75 73.66 0)
+    (property "Footprint" "Resistor_SMD:R_01005_0402Metric" (at 158.75 73.66 0)
       (effects (font (size 1.27 1.27)) hide)
     )
@@
       (effects (font (size 1.27 1.27)))
     )
-    (property "Footprint" "" (at 125.73 104.14 0)
+    (property "Footprint" "Resistor_SMD:R_01005_0402Metric" (at 125.73 104.14 0)
       (effects (font (size 1.27 1.27)) hide)
     )
@@
     )
   )
+  (symbol (lib_id "power:GND") (at 212.09 114.3 270) (unit 1)
+    (in_bom yes) (on_board yes) (dnp no) (fields_autoplaced)
+    (property "Reference" "#PWR010" (at 205.74 114.3 0)
+      (effects (font (size 1.27 1.27)) hide)
+    )
+    (property "Value" "GND" (at 208.28 114.3 90)
+      (effects (font (size 1.27 1.27)) (justify right))
+    )
+    (property "Footprint" "" (at 212.09 114.3 0)
+      (effects (font (size 1.27 1.27)) hide)
+    )
+    (property "Datasheet" "" (at 212.09 114.3 0)
+      (effects (font (size 1.27 1.27)) hide)
+    )
+    (pin "1")
+    (instances
+      (project "bno085-i2c-board"
+        (path "/a6bdf641-e64e-4bd0-89ab-89241b3a6e60"
+          (reference "#PWR010") (unit 1)
+        )
+      )
+    )
+  )
   (symbol (lib_id "Device:R_Small") (at 176.53 120.65 0) (unit 1)
     (in_bom yes) (on_board yes) (dnp no) (fields_autoplaced)
@@
       (effects (font (size 1.27 1.27)) (justify left))
     )
-    (property "Footprint" "" (at 176.53 120.65 0)
+    (property "Footprint" "Resistor_SMD:R_01005_0402Metric" (at 176.53 120.65 0)
       (effects (font (size 1.27 1.27)) hide)
     )
@@
       (effects (font (size 1.27 1.27)))
     )
-    (property "Footprint" "" (at 149.86 93.98 0)
+    (property "Footprint" "Package_LGA:LGA-28_5.2x3.8mm_P0.5mm" (at 149.86 93.98 0)
       (effects (font (size 1.27 1.27)) hide)
     )
@@
       (effects (font (size 1.27 1.27)))
     )
-    (property "Footprint" "" (at 172.72 104.14 0)
+    (property "Footprint" "Resistor_SMD:R_01005_0402Metric" (at 172.72 104.14 0)
       (effects (font (size 1.27 1.27)) hide)
     )
@@
     )
   )
-  (symbol (lib_id "power:GND") (at 212.09 104.14 270) (unit 1)
-    (in_bom yes) (on_board yes) (dnp no) (fields_autoplaced)
-    (property "Reference" "#PWR010" (at 205.74 104.14 0)
-      (effects (font (size 1.27 1.27)) hide)
-    )
-    (property "Value" "GND" (at 208.28 104.14 90)
-      (effects (font (size 1.27 1.27)) (justify right))
-    )
-    (property "Footprint" "" (at 212.09 104.14 0)
-      (effects (font (size 1.27 1.27)) hide)
-    )
-    (property "Datasheet" "" (at 212.09 104.14 0)
-      (effects (font (size 1.27 1.27)) hide)
-    )
-    (pin "1")
-    (instances
-      (project "bno085-i2c-board"
-        (path "/a6bdf641-e64e-4bd0-89ab-89241b3a6e60"
-          (reference "#PWR010") (unit 1)
-        )
-      )
-    )
-  )
   (symbol (lib_id "power:+3.3V") (at 132.08 91.44 90) (unit 1)
     (in_bom yes) (on_board yes) (dnp no)
@@
     )
   )
-  (symbol (lib_id "power:+3.3V") (at 207.01 101.6 90) (unit 1)
-    (in_bom yes) (on_board yes) (dnp no) (fields_autoplaced)
-    (property "Reference" "#PWR012" (at 210.82 101.6 0)
-      (effects (font (size 1.27 1.27)) hide)
-    )
-    (property "Value" "+3.3V" (at 203.2 101.6 90)
-      (effects (font (size 1.27 1.27)) (justify left))
-    )
-    (property "Footprint" "" (at 207.01 101.6 0)
-      (effects (font (size 1.27 1.27)) hide)
-    )
-    (property "Datasheet" "" (at 207.01 101.6 0)
+  (symbol (lib_id "power:+3.3V") (at 209.55 111.76 90) (unit 1)
+    (in_bom yes) (on_board yes) (dnp no) (fields_autoplaced)
+    (property "Reference" "#PWR012" (at 213.36 111.76 0)
+      (effects (font (size 1.27 1.27)) hide)
+    )
+    (property "Value" "+3.3V" (at 205.74 111.76 90)
+      (effects (font (size 1.27 1.27)) (justify left))
+    )
+    (property "Footprint" "" (at 209.55 111.76 0)
+      (effects (font (size 1.27 1.27)) hide)
+    )
+    (property "Datasheet" "" (at 209.55 111.76 0)
       (effects (font (size 1.27 1.27)) hide)
     )
@@
       (effects (font (size 1.27 1.27)))
     )
-    (property "Footprint" "" (at 146.05 128.27 0)
+    (property "Footprint" "Resistor_SMD:R_01005_0402Metric" (at 146.05 128.27 0)
       (effects (font (size 1.27 1.27)) hide)
     )
@@
       (effects (font (size 1.27 1.27)) (justify right))
     )
-    (property "Footprint" "" (at 217.17 109.22 0)
-      (effects (font (size 1.27 1.27)) hide)
-    )
+    (property "Footprint" "Connector_PinHeader_2.54mm:PinHeader_1x06_P2.54mm_Horizontal" (at 217.17 109.22 0)
+      (effects (font (size 1.27 1.27)) hide)
+    )

Commit message: new pcb resistors
Parts:
- R1, R2, R3, R4, R5: footprint Resistor_SMD:R_01005_0402Metric -> Resistor_SMD:R_0805_2012Metric
Connections:
- net +3.3V: now also R5.2
- net H_SDA: now also U1.20 (H_SDA/H_MISO/TX)
Other:
- moved on the sheet: R5
Changed lines of the file:
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@@
   (junction (at 132.08 73.66) (diameter 0) (color 0 0 0 0)
+  )
+  (junction (at 176.53 104.14) (diameter 0) (color 0 0 0 0)
   )
   (junction (at 212.09 111.76) (diameter 0) (color 0 0 0 0)
@@
     (stroke (width 0) (type default))
   )
-  (wire (pts (xy 167.64 104.14) (xy 170.18 104.14))
-    (stroke (width 0) (type default))
-  )
   (wire (pts (xy 132.08 115.57) (xy 129.54 115.57))
     (stroke (width 0) (type default))
@@
     (stroke (width 0) (type default))
   )
+  (wire (pts (xy 176.53 104.14) (xy 180.34 104.14))
+    (stroke (width 0) (type default))
+  )
   (wire (pts (xy 182.88 114.3) (xy 176.53 114.3))
     (stroke (width 0) (type default))
@@
     (stroke (width 0) (type default))
   )
+  (wire (pts (xy 176.53 111.76) (xy 176.53 114.3))
+    (stroke (width 0) (type default))
+  )
   (wire (pts (xy 119.38 104.14) (xy 123.19 104.14))
     (stroke (width 0) (type default))
@@
     (stroke (width 0) (type default))
   )
+  (wire (pts (xy 176.53 104.14) (xy 176.53 106.68))
+    (stroke (width 0) (type default))
+  )
   (wire (pts (xy 119.38 93.98) (xy 132.08 93.98))
     (stroke (width 0) (type default))
@@
     (stroke (width 0) (type default))
   )
-  (wire (pts (xy 175.26 104.14) (xy 180.34 104.14))
+  (wire (pts (xy 167.64 104.14) (xy 176.53 104.14))
     (stroke (width 0) (type default))
   )
@@
       (effects (font (size 1.27 1.27)))
     )
-    (property "Footprint" "Resistor_SMD:R_01005_0402Metric" (at 158.75 73.66 0)
+    (property "Footprint" "Resistor_SMD:R_0805_2012Metric" (at 158.75 73.66 0)
       (effects (font (size 1.27 1.27)) hide)
     )
@@
       (effects (font (size 1.27 1.27)))
     )
-    (property "Footprint" "Resistor_SMD:R_01005_0402Metric" (at 125.73 104.14 0)
+    (property "Footprint" "Resistor_SMD:R_0805_2012Metric" (at 125.73 104.14 0)
       (effects (font (size 1.27 1.27)) hide)
     )
@@
       (effects (font (size 1.27 1.27)) (justify left))
     )
-    (property "Footprint" "Resistor_SMD:R_01005_0402Metric" (at 176.53 120.65 0)
+    (property "Footprint" "Resistor_SMD:R_0805_2012Metric" (at 176.53 120.65 0)
       (effects (font (size 1.27 1.27)) hide)
     )
@@
     )
   )
-  (symbol (lib_id "Device:R_Small") (at 172.72 104.14 270) (unit 1)
-    (in_bom yes) (on_board yes) (dnp no)
-    (property "Reference" "R5" (at 172.72 109.22 90)
-      (effects (font (size 1.27 1.27)))
-    )
-    (property "Value" "2.2k" (at 172.72 106.68 90)
-      (effects (font (size 1.27 1.27)))
-    )
-    (property "Footprint" "Resistor_SMD:R_01005_0402Metric" (at 172.72 104.14 0)
-      (effects (font (size 1.27 1.27)) hide)
-    )
-    (property "Datasheet" "~" (at 172.72 104.14 0)
+  (symbol (lib_id "Device:R_Small") (at 176.53 109.22 0) (unit 1)
+    (in_bom yes) (on_board yes) (dnp no)
+    (property "Reference" "R5" (at 181.61 109.22 90)
+      (effects (font (size 1.27 1.27)))
+    )
+    (property "Value" "2.2k" (at 179.07 109.22 90)
+      (effects (font (size 1.27 1.27)))
+    )
+    (property "Footprint" "Resistor_SMD:R_0805_2012Metric" (at 176.53 109.22 0)
+      (effects (font (size 1.27 1.27)) hide)
+    )
+    (property "Datasheet" "~" (at 176.53 109.22 0)
       (effects (font (size 1.27 1.27)) hide)
     )
@@
       (effects (font (size 1.27 1.27)))
     )
-    (property "Footprint" "Resistor_SMD:R_01005_0402Metric" (at 146.05 128.27 0)
-      (effects (font (size 1.27 1.27)) hide)
-    )
+    (property "Footprint" "Resistor_SMD:R_0805_2012Metric" (at 146.05 128.27 0)
+      (effects (font (size 1.27 1.27)) hide)
+    )

Commit message: pcb
Other:
- title: (none) -> BNO085 I2C Board
Changed lines of the file:
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@@
 (kicad_sch (version 20230121) (generator eeschema)
   (paper "A4")
+  (title_block
+    (title "BNO085 I2C Board")
+    (date "2023-06-22")
+  )
   (junction (at 176.53 124.46) (diameter 0) (color 0 0 0 0)
   )
