File: hardware/bno085-i2c-board-v2/bno085-i2c-board-v2.kicad_sch (KiCad schematic)
At the start: 8 parts, among them J1 Conn_01x06_Pin

Commit message: new board
Parts:
- removed J1: Conn_01x06_Pin, Connector_PinHeader_2.54mm:PinHeader_1x06_P2.54mm_Horizontal, symbol Connector:Conn_01x06_Pin
- added J1, J2, J3, J4, J5, J6: Conn_01x01_Pin, Connector_PinHeader_2.54mm:PinHeader_1x01_P2.54mm_Vertical, symbol Connector:Conn_01x01_Pin
- C1: footprint Capacitor_SMD:CP_Elec_4x3.9 -> Capacitor_SMD:C_0402_1005Metric
- R1, R2, R3, R4, R5: footprint Resistor_SMD:R_0805_2012Metric -> Resistor_SMD:R_0402_1005Metric
Connections:
- net +3.3V: now also J6.1 (Pin_1)
- net GND: now also J5.1 (Pin_1)
- net H_INTN: no longer names the net of U1.14 (H_INTN)
- net H_INTN: now also J1.1 (Pin_1)
- net H_SCL: no longer names the net of R4.2, U1.19 (H_SCL/SCK/RX)
- net H_SCL: now also J4.1 (Pin_1)
- net H_SDA: no longer names the net of R5.1, U1.20 (H_SDA/H_MISO/TX)
- net H_SDA: now also J3.1 (Pin_1)
- net NRST: no longer names the net of U1.11 (NRST)
- net NRST: now also J2.1 (Pin_1)
Other:
- title: BNO085 I2C Board -> (none)

Commit message: round board
Parts:
- J1, J2, J3, J4, J5, J6: footprint Connector_PinHeader_2.54mm:PinHeader_1x01_P2.54mm_Vertical -> Connector_PinHeader_1.00mm:PinHeader_1x01_P1.00mm_Vertical
Changed lines of the file:
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@@
       (effects (font (size 1.27 1.27)))
     )
-    (property "Footprint" "Connector_PinHeader_2.54mm:PinHeader_1x01_P2.54mm_Vertical" (at 185.42 104.14 0)
+    (property "Footprint" "Connector_PinHeader_1.00mm:PinHeader_1x01_P1.00mm_Vertical" (at 185.42 104.14 0)
       (effects (font (size 1.27 1.27)) hide)
     )
@@
       (effects (font (size 1.27 1.27)))
     )
-    (property "Footprint" "Connector_PinHeader_2.54mm:PinHeader_1x01_P2.54mm_Vertical" (at 193.04 124.46 0)
+    (property "Footprint" "Connector_PinHeader_1.00mm:PinHeader_1x01_P1.00mm_Vertical" (at 193.04 124.46 0)
       (effects (font (size 1.27 1.27)) hide)
     )
@@
       (effects (font (size 1.27 1.27)))
     )
-    (property "Footprint" "Connector_PinHeader_2.54mm:PinHeader_1x01_P2.54mm_Vertical" (at 114.3 93.98 0)
+    (property "Footprint" "Connector_PinHeader_1.00mm:PinHeader_1x01_P1.00mm_Vertical" (at 114.3 93.98 0)
       (effects (font (size 1.27 1.27)) hide)
     )
@@
       (effects (font (size 1.27 1.27)))
     )
-    (property "Footprint" "Connector_PinHeader_2.54mm:PinHeader_1x01_P2.54mm_Vertical" (at 217.17 114.3 0)
+    (property "Footprint" "Connector_PinHeader_1.00mm:PinHeader_1x01_P1.00mm_Vertical" (at 217.17 114.3 0)
       (effects (font (size 1.27 1.27)) hide)
     )
@@
       (effects (font (size 1.27 1.27)))
     )
-    (property "Footprint" "Connector_PinHeader_2.54mm:PinHeader_1x01_P2.54mm_Vertical" (at 114.3 101.6 0)
+    (property "Footprint" "Connector_PinHeader_1.00mm:PinHeader_1x01_P1.00mm_Vertical" (at 114.3 101.6 0)
       (effects (font (size 1.27 1.27)) hide)
     )
@@
       (effects (font (size 1.27 1.27)))
     )
-    (property "Footprint" "Connector_PinHeader_2.54mm:PinHeader_1x01_P2.54mm_Vertical" (at 217.17 111.76 0)
-      (effects (font (size 1.27 1.27)) hide)
-    )
+    (property "Footprint" "Connector_PinHeader_1.00mm:PinHeader_1x01_P1.00mm_Vertical" (at 217.17 111.76 0)
+      (effects (font (size 1.27 1.27)) hide)
+    )
