File: hardware/bno085-i2c-board-v3/bno085-i2c-board-v3.kicad_sch (KiCad schematic)
At the start: 11 parts, among them J3 Conn_01x01_Pin, J4 Conn_01x01_Pin, J5 Conn_01x01_Pin, J6 Conn_01x01_Pin

Commit message: metadata
Other:
- title: (none) -> BNO085-I2C Interface Board
Changed lines of the file:
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@@
 (kicad_sch (version 20230121) (generator eeschema)
   (paper "A4")
+  (title_block
+    (title "BNO085-I2C Interface Board")
+    (date "2023-06-27")
+  )
   (junction (at 176.53 124.46) (diameter 0) (color 0 0 0 0)
   )
