File: hardware/bno085-i2c-board-v3/bno085-i2c-board-v3.kicad_pcb (KiCad board)
At the start: 2 copper layers, 10 x 10 mm, 11 parts, among them J1 Conn_01x01_Pin, J2 Conn_01x01_Pin, J3 Conn_01x01_Pin, J4 Conn_01x01_Pin

Commit message: added key
Other:
- outline, holes or cut-outs redrawn
Changed lines of the file:
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@@
     )
   )
-  (gr_circle (center 167.5 97.5) (end 172.5 97.5)
-    (stroke (width 0.1) (type default)) (fill none) (layer "Edge.Cuts"))
+  (gr_arc (start 165.469307 92.930942) (mid 164.621614 94.621614) (end 162.930942 95.469307)
+    (stroke (width 0.1) (type default)) (layer "Edge.Cuts"))
+  (gr_arc (start 167.5 92.5) (mid 170.224568 101.692461) (end 162.930942 95.469308)
+    (stroke (width 0.1) (type default)) (layer "Edge.Cuts"))
+  (gr_arc (start 165.469308 92.930942) (mid 166.462043 92.608922) (end 167.5 92.5)
+    (stroke (width 0.1) (type default)) (layer "Edge.Cuts"))
   (gr_text "3V3" (at 163.853651 96.667677 270) (layer "F.SilkS")
     (effects (font (size 0.6 0.6) (thickness 0.1) bold) (justify left bottom))

Commit message: jlc fab files
Other:
- board text added: "DO NOT USE THIS DESIGN USE V3-PANEL-BASE"
Changed lines of the file:
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@@
     (effects (font (size 0.6 0.6) (thickness 0.1) bold) (justify left bottom))
   )
-  (dimension (type orthogonal) (layer "Cmts.User")
+  (gr_text "DO NOT USE THIS DESIGN\nUSE V3-PANEL-BASE" (at 154.94 99.06) (layer "Cmts.User")
+    (effects (font (size 1.5 1.5) (thickness 0.3) bold) (justify left bottom))
+  )
+  (dimension (type orthogonal) (layer "Dwgs.User")
     (pts (xy 162.5 97.5) (xy 172.5 97.5))
     (height -7.5)
     (orientation 0)
-    (gr_text "10.0000 mm" (at 167.5 88.85) (layer "Cmts.User")
+    (gr_text "10.0000 mm" (at 167.5 88.85) (layer "Dwgs.User")
       (effects (font (size 1 1) (thickness 0.15)))
     )
