File: hardware/bno085-i2c-board-v3-panel/bno085-i2c-board-v3-panel.kicad_pcb (KiCad board)
At the start: 2 copper layers, 72 x 72 mm, 631 parts, among them J1 Conn_01x01_Pin, J2 Conn_01x01_Pin, J3 Conn_01x01_Pin, J4 Conn_01x01_Pin

Commit message: small panels
Other:
- board text added: "BNO085 Interface Board | 2023-06-30"
- board text removed: "|"
