File: hardware/bno085-i2c-board-v3-square/bno085-i2c-board-v3-square.kicad_pcb (KiCad board)
At the start: 2 copper layers, 8 x 11.3 mm, 8 parts, among them J5 Conn_01x04_Pin

Commit message: square panel
Changed lines of the file:
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@@
     (property "ki_keywords" "connector")
     (attr through_hole)
-    (fp_text reference "J5" (at 4.464917 1.490663 180) (layer "F.SilkS")
+    (fp_text reference "J5" (at 4.464917 1.490663 180) (layer "F.SilkS") hide
         (effects (font (size 1 1) (thickness 0.15)))
     )
