File: hardware/bno085-i2c-board-v3-large/bno085-i2c-board-v3-large.kicad_sch (KiCad schematic)
At the start: 11 parts, among them J1 Conn_01x01_Pin, J2 Conn_01x01_Pin, J3 Conn_01x01_Pin, J4 Conn_01x01_Pin

Commit message: c
Parts:
- U1: value ~ -> BNO08x
Other:
- moved on the sheet: R5
Changed lines of the file:
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@@
 (kicad_sch (version 20230121) (generator eeschema)
   (paper "A4")
-  (junction (at 176.53 124.46) (diameter 0) (color 0 0 0 0)
-  )
   (junction (at 170.18 114.3) (diameter 0) (color 0 0 0 0)
   )
@@
   )
   (junction (at 132.08 73.66) (diameter 0) (color 0 0 0 0)
+  )
+  (junction (at 173.99 124.46) (diameter 0) (color 0 0 0 0)
+  )
+  (junction (at 173.99 114.3) (diameter 0) (color 0 0 0 0)
   )
   (junction (at 176.53 104.14) (diameter 0) (color 0 0 0 0)
@@
     (stroke (width 0) (type default))
   )
-  (wire (pts (xy 176.53 124.46) (xy 187.96 124.46))
-    (stroke (width 0) (type default))
-  )
   (wire (pts (xy 132.08 73.66) (xy 148.59 73.66))
     (stroke (width 0) (type default))
   )
-  (wire (pts (xy 176.53 123.19) (xy 176.53 124.46))
+  (wire (pts (xy 173.99 123.19) (xy 173.99 124.46))
     (stroke (width 0) (type default))
   )
@@
     (stroke (width 0) (type default))
   )
+  (wire (pts (xy 173.99 114.3) (xy 170.18 114.3))
+    (stroke (width 0) (type default))
+  )
   (wire (pts (xy 119.38 104.14) (xy 123.19 104.14))
     (stroke (width 0) (type default))
@@
     (stroke (width 0) (type default))
   )
-  (wire (pts (xy 153.67 124.46) (xy 176.53 124.46))
+  (wire (pts (xy 153.67 124.46) (xy 173.99 124.46))
     (stroke (width 0) (type default))
   )
@@
     (stroke (width 0) (type default))
   )
-  (wire (pts (xy 176.53 114.3) (xy 176.53 118.11))
-    (stroke (width 0) (type default))
-  )
-  (wire (pts (xy 176.53 114.3) (xy 170.18 114.3))
+  (wire (pts (xy 173.99 114.3) (xy 173.99 118.11))
+    (stroke (width 0) (type default))
+  )
+  (wire (pts (xy 173.99 124.46) (xy 187.96 124.46))
+    (stroke (width 0) (type default))
+  )
+  (wire (pts (xy 176.53 114.3) (xy 173.99 114.3))
     (stroke (width 0) (type default))
   )
@@
     (pin "1")
     (instances
-      (project "bno085-i2c-board-v3"
-        (path "/91467fd9-c59b-4cd8-a593-aab0738bbb6c"
+      (project "bno085-i2c-board-v3-large"
+        (path "/65945718-ecdd-4a51-8bb6-fdef4c66336c"
           (reference "#PWR04") (unit 1)
         )
       )
+      (project "bno085-i2c-board-v3"
+        (path "/91467fd9-c59b-4cd8-a593-aab0738bbb6c"
+          (reference "#PWR04") (unit 1)
+        )
+      )
       (project "bno085-i2c-board-v2"
         (path "/9217d116-cf40-485a-abd0-8ce710fa4b1d"
@@
     (pin "1")
     (instances
-      (project "bno085-i2c-board-v3"
-        (path "/91467fd9-c59b-4cd8-a593-aab0738bbb6c"
+      (project "bno085-i2c-board-v3-large"
+        (path "/65945718-ecdd-4a51-8bb6-fdef4c66336c"
           (reference "#PWR07") (unit 1)
         )
       )
+      (project "bno085-i2c-board-v3"
+        (path "/91467fd9-c59b-4cd8-a593-aab0738bbb6c"
+          (reference "#PWR07") (unit 1)
+        )
+      )
       (project "bno085-i2c-board-v2"
         (path "/9217d116-cf40-485a-abd0-8ce710fa4b1d"
@@
     (pin "1")
     (instances
+      (project "bno085-i2c-board-v3-large"
+        (path "/65945718-ecdd-4a51-8bb6-fdef4c66336c"
+          (reference "#PWR06") (unit 1)
+        )
+      )
       (project "bno085-i2c-board-v3"
         (path "/91467fd9-c59b-4cd8-a593-aab0738bbb6c"
@@
     (pin "1")
     (instances
-      (project "bno085-i2c-board-v3"
-        (path "/91467fd9-c59b-4cd8-a593-aab0738bbb6c"
+      (project "bno085-i2c-board-v3-large"
+        (path "/65945718-ecdd-4a51-8bb6-fdef4c66336c"
           (reference "#PWR012") (unit 1)
         )
       )
+      (project "bno085-i2c-board-v3"
+        (path "/91467fd9-c59b-4cd8-a593-aab0738bbb6c"
+          (reference "#PWR012") (unit 1)
+        )
+      )
       (project "bno085-i2c-board-v2"
         (path "/9217d116-cf40-485a-abd0-8ce710fa4b1d"
@@
     )
   )
-  (symbol (lib_id "Device:R_Small") (at 176.53 120.65 0) (unit 1)
-    (in_bom yes) (on_board yes) (dnp no) (fields_autoplaced)
-    (property "Reference" "R5" (at 179.07 119.38 0)
+  (symbol (lib_id "Device:R_Small") (at 173.99 120.65 0) (unit 1)
+    (in_bom yes) (on_board yes) (dnp no) (fields_autoplaced)
+    (property "Reference" "R5" (at 176.53 119.38 0)
       (effects (font (size 1.27 1.27)) (justify left))
     )
-    (property "Value" "2.2k" (at 179.07 121.92 0)
+    (property "Value" "2.2k" (at 176.53 121.92 0)
       (effects (font (size 1.27 1.27)) (justify left))
     )
-    (property "Footprint" "Resistor_SMD:R_0402_1005Metric" (at 176.53 120.65 0)
-      (effects (font (size 1.27 1.27)) hide)
-    )
-    (property "Datasheet" "~" (at 176.53 120.65 0)
+    (property "Footprint" "Resistor_SMD:R_0402_1005Metric" (at 173.99 120.65 0)
+      (effects (font (size 1.27 1.27)) hide)
+    )
+    (property "Datasheet" "~" (at 173.99 120.65 0)
       (effects (font (size 1.27 1.27)) hide)
     )
@@
       (effects (font (size 1.27 1.27)) (justify left))
     )
-    (property "Value" "~" (at 149.86 93.98 0)
+    (property "Value" "BNO08x" (at 149.86 93.98 0)
       (effects (font (size 1.27 1.27)))
     )
@@
     (pin "1")
     (instances
+      (project "bno085-i2c-board-v3-large"
+        (path "/65945718-ecdd-4a51-8bb6-fdef4c66336c"
+          (reference "#PWR09") (unit 1)
+        )
+      )
       (project "bno085-i2c-board-v3"
         (path "/91467fd9-c59b-4cd8-a593-aab0738bbb6c"
@@
     (pin "1")
     (instances
+      (project "bno085-i2c-board-v3-large"
+        (path "/65945718-ecdd-4a51-8bb6-fdef4c66336c"
+          (reference "#PWR02") (unit 1)
+        )
+      )
       (project "bno085-i2c-board-v3"
         (path "/91467fd9-c59b-4cd8-a593-aab0738bbb6c"
@@
     (pin "1")
     (instances
+      (project "bno085-i2c-board-v3-large"
+        (path "/65945718-ecdd-4a51-8bb6-fdef4c66336c"
+          (reference "#PWR08") (unit 1)
+        )
+      )
       (project "bno085-i2c-board-v3"
         (path "/91467fd9-c59b-4cd8-a593-aab0738bbb6c"
@@
     (pin "1")
     (instances
+      (project "bno085-i2c-board-v3-large"
+        (path "/65945718-ecdd-4a51-8bb6-fdef4c66336c"
+          (reference "#PWR010") (unit 1)
+        )
+      )
       (project "bno085-i2c-board-v3"
         (path "/91467fd9-c59b-4cd8-a593-aab0738bbb6c"
@@
     (pin "1")
     (instances
+      (project "bno085-i2c-board-v3-large"
+        (path "/65945718-ecdd-4a51-8bb6-fdef4c66336c"
+          (reference "#PWR05") (unit 1)
+        )
+      )
       (project "bno085-i2c-board-v3"
         (path "/91467fd9-c59b-4cd8-a593-aab0738bbb6c"
@@
     (pin "1")
     (instances
+      (project "bno085-i2c-board-v3-large"
+        (path "/65945718-ecdd-4a51-8bb6-fdef4c66336c"
+          (reference "#PWR011") (unit 1)
+        )
+      )
       (project "bno085-i2c-board-v3"
         (path "/91467fd9-c59b-4cd8-a593-aab0738bbb6c"
@@
     (pin "1")
     (instances
+      (project "bno085-i2c-board-v3-large"
+        (path "/65945718-ecdd-4a51-8bb6-fdef4c66336c"
+          (reference "#PWR01") (unit 1)
+        )
+      )
       (project "bno085-i2c-board-v3"
         (path "/91467fd9-c59b-4cd8-a593-aab0738bbb6c"
@@
     (pin "1")
     (instances
-      (project "bno085-i2c-board-v3"
-        (path "/91467fd9-c59b-4cd8-a593-aab0738bbb6c"
+      (project "bno085-i2c-board-v3-large"
+        (path "/65945718-ecdd-4a51-8bb6-fdef4c66336c"
+          (reference "#PWR03") (unit 1)
+        )
+      )
+      (project "bno085-i2c-board-v3"
+        (path "/91467fd9-c59b-4cd8-a593-aab0738bbb6c"
