File: hardware/bno085-i2c-board-v4-large/bno085-i2c-board-v4-large.kicad_pcb (KiCad board)
At the start: 2 copper layers, 16 x 16 mm, 11 parts, among them J1 Conn_01x01_Pin, J2 Conn_01x01_Pin, J3 Conn_01x01_Pin, J4 Conn_01x01_Pin

Commit message: panels
Changed lines of the file:
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@@
     (property "Sheetname" "")
     (attr smd)
-    (fp_text reference "U1" (at -1.28 -0.94) (layer "F.SilkS")
+    (fp_text reference "U1" (at 0 0) (layer "F.SilkS")
         (effects (font (size 1 1) (thickness 0.15)))
     )
