File: hardware/bno085-i2c-board-v4-large-panel/bno085-i2c-board-v4-large-panel.kicad_pcb (KiCad board)
At the start: 2 copper layers, 102 x 102 mm, 437 parts, among them J1 Conn_01x01_Pin, J2 Conn_01x01_Pin, J3 Conn_01x01_Pin, J4 Conn_01x01_Pin

Commit message: v4-large-panel
Parts:
- removed the REF** at (130.5, 80.9)
- removed the REF** at (130.5, 115.1)
- removed the REF** at (192.6, 71.0)
- removed the REF** at (100.0, 22.5) (x2)
- removed the REF** at (192.6, 53.0)
- removed the REF** at (174.6, 89.0)
- removed the REF** at (192.6, 107.0)
- removed the REF** at (184.5, 44.9)
- removed the REF** at (176.4, 89.0)
- removed the REF** at (148.5, 80.9)
- removed the REF** at (148.5, 79.1)
- removed the REF** at (148.5, 62.9)
- removed the REF** at (138.6, 35.0)
- removed the REF** at (130.5, 98.9)
- removed the REF** at (148.5, 98.9)
- removed the REF** at (122.4, 53.0)
- removed the REF** at (138.6, 89.0)
- removed the REF** at (104.4, 89.0)
- removed the REF** at (112.5, 79.1)
- removed the REF** at (158.4, 89.0)
- removed the REF** at (166.5, 61.1)
- removed the REF** at (130.5, 61.1)
- removed the REF** at (156.6, 89.0)
- removed the REF** at (120.6, 53.0)
- removed the REF** at (166.5, 43.1)
- removed the REF** at (112.5, 61.1)
- removed the REF** at (148.5, 43.1)
- removed the REF** at (148.5, 115.1)
- removed the REF** at (184.5, 61.1)
- removed the REF** at (184.5, 26.9)
- removed the REF** at (192.6, 35.0)
- removed the REF** at (140.4, 107.0)
- removed the REF** at (112.5, 115.1)
- removed the REF** at (148.5, 26.9)
- removed the REF** at (130.5, 79.1)
- removed the REF** at (138.6, 107.0)
- removed the REF** at (112.5, 62.9)
- removed the REF** at (148.5, 97.1)
- removed the REF** at (112.5, 43.1)
- removed the REF** at (140.4, 35.0)
- removed the REF** at (112.5, 80.9)
- removed the REF** at (148.5, 61.1)
- removed the REF** at (184.5, 79.1)
- removed the REF** at (166.5, 98.9)
- removed the REF** at (156.6, 107.0)
- removed the REF** at (197.0, 22.5) (x2)
- removed the REF** at (100.0, 119.5) (x2)
- removed the REF** at (130.5, 26.9)
- removed the REF** at (120.6, 71.0)
- removed the REF** at (130.5, 44.9)
- removed the REF** at (174.6, 71.0)
- removed the REF** at (148.5, 44.9)
- removed the REF** at (174.6, 107.0)
- removed the REF** at (104.4, 107.0)
- removed the REF** at (130.5, 62.9)
- removed the REF** at (166.5, 26.9)
- removed the REF** at (122.4, 89.0)
- removed the REF** at (166.5, 80.9)
- removed the REF** at (120.6, 35.0)
- removed the REF** at (176.4, 71.0)
- removed the REF** at (156.6, 35.0)
- removed the REF** at (104.4, 71.0)
- removed the REF** at (166.5, 79.1)
- removed the REF** at (156.6, 53.0)
- removed the REF** at (174.6, 35.0)
- removed the REF** at (112.5, 44.9)
- removed the REF** at (104.4, 53.0)
- removed the REF** at (158.4, 71.0)
- removed the REF** at (176.4, 53.0)
- removed the REF** at (112.5, 26.9)
- removed the REF** at (122.4, 71.0)
- removed the REF** at (158.4, 53.0)
- removed the REF** at (166.5, 62.9)
- removed the REF** at (184.5, 80.9)
- removed the REF** at (120.6, 107.0)
- removed the REF** at (174.6, 53.0)
- removed the REF** at (122.4, 35.0)
- removed the REF** at (122.4, 107.0)
- removed the REF** at (184.5, 43.1)
- removed the REF** at (192.6, 89.0)
- removed the REF** at (166.5, 97.1)
- removed the REF** at (130.5, 97.1)
- removed the REF** at (138.6, 71.0)
- removed the REF** at (156.6, 71.0)
- removed the REF** at (184.5, 97.1)
- removed the REF** at (184.5, 115.1)
- removed the REF** at (158.4, 107.0)
- removed the REF** at (138.6, 53.0)
- removed the REF** at (184.5, 62.9)
- removed the REF** at (112.5, 98.9)
- removed the REF** at (130.5, 43.1)
- removed the REF** at (176.4, 107.0)
- removed the REF** at (120.6, 89.0)
- removed the REF** at (166.5, 44.9)
- removed the REF** at (140.4, 53.0)
- removed the REF** at (140.4, 89.0)
- removed the REF** at (184.5, 98.9)
- removed the REF** at (140.4, 71.0)
- removed the REF** at (166.5, 115.1)
- removed the REF** at (112.5, 97.1)
- added REF**: NPTH, NPTH, F.Cu at (156.6, 88.2)
- added REF**: NPTH, NPTH, F.Cu at (112.5, 62.9)
- added REF**: NPTH, NPTH, F.Cu at (147.7, 79.1)
- added REF**: NPTH, NPTH, F.Cu at (184.5, 43.1)
- added REF**: NPTH, NPTH, F.Cu at (158.4, 34.2)
- added REF**: NPTH, NPTH, F.Cu at (174.6, 106.2)
- added REF**: Fiducial, Fiducial, F.Cu at (197.0, 22.5)
- added REF**: NPTH, NPTH, F.Cu at (192.6, 88.2)
- added REF**: NPTH, NPTH, F.Cu at (140.4, 107.0)
- added REF**: NPTH, NPTH, F.Cu at (130.5, 97.1)
- added REF**: NPTH, NPTH, F.Cu at (104.4, 89.8)
- added REF**: NPTH, NPTH, F.Cu at (122.4, 35.8)
- added REF**: NPTH, NPTH, F.Cu at (167.3, 43.1)
- added REF**: NPTH, NPTH, F.Cu at (111.7, 80.9)
- added REF**: NPTH, NPTH, F.Cu at (148.5, 80.9)
- added REF**: NPTH, NPTH, F.Cu at (148.5, 79.1)
- added REF**: NPTH, NPTH, F.Cu at (184.5, 62.9)
- added REF**: NPTH, NPTH, F.Cu at (130.5, 79.1)
- added REF**: NPTH, NPTH, F.Cu at (113.3, 43.1)
- added REF**: NPTH, NPTH, F.Cu at (158.4, 35.8)
- added REF**: NPTH, NPTH, F.Cu at (138.6, 89.8)
- added REF**: NPTH, NPTH, F.Cu at (138.6, 53.0)
- added REF**: NPTH, NPTH, F.Cu at (166.5, 80.9)
- added REF**: NPTH, NPTH, F.Cu at (112.5, 115.1)
- added REF**: NPTH, NPTH, F.Cu at (176.4, 71.8)
- added REF**: NPTH, NPTH, F.Cu at (131.3, 115.1)
- added REF**: NPTH, NPTH, F.Cu at (149.3, 26.9)
- added REF**: NPTH, NPTH, F.Cu at (165.7, 79.1)
- added REF**: NPTH, NPTH, F.Cu at (131.3, 43.1)
- added REF**: NPTH, NPTH, F.Cu at (166.5, 43.1)
- added REF**: NPTH, NPTH, F.Cu at (138.6, 35.8)
- added REF**: NPTH, NPTH, F.Cu at (113.3, 98.9)
- added REF**: NPTH, NPTH, F.Cu at (192.6, 53.8)
- added REF**: NPTH, NPTH, F.Cu at (129.7, 79.1)
- added REF**: NPTH, NPTH, F.Cu at (174.6, 52.2)
- added REF**: NPTH, NPTH, F.Cu at (165.7, 44.9)
- added REF**: NPTH, NPTH, F.Cu at (130.5, 43.1)
- added REF**: NPTH, NPTH, F.Cu at (104.4, 53.0)
- added REF**: NPTH, NPTH, F.Cu at (129.7, 80.9)
- added REF**: NPTH, NPTH, F.Cu at (176.4, 35.8)
- added REF**: NPTH, NPTH, F.Cu at (122.4, 106.2)
- added REF**: NPTH, NPTH, F.Cu at (192.6, 106.2)
- added REF**: NPTH, NPTH, F.Cu at (158.4, 70.2)
- added REF**: NPTH, NPTH, F.Cu at (156.6, 35.0)
- added REF**: NPTH, NPTH, F.Cu at (176.4, 107.0)
- added REF**: NPTH, NPTH, F.Cu at (148.5, 26.9)
- added REF**: NPTH, NPTH, F.Cu at (147.7, 62.9)
- added REF**: NPTH, NPTH, F.Cu at (140.4, 89.0)
- added REF**: NPTH, NPTH, F.Cu at (138.6, 88.2)
- added REF**: NPTH, NPTH, F.Cu at (104.4, 34.2)
- added REF**: NPTH, NPTH, F.Cu at (140.4, 35.8)
- added REF**: NPTH, NPTH, F.Cu at (129.7, 115.1)
- added REF**: NPTH, NPTH, F.Cu at (120.6, 52.2)
- added REF**: NPTH, NPTH, F.Cu at (140.4, 88.2)
- added REF**: NPTH, NPTH, F.Cu at (120.6, 88.2)
- added REF**: NPTH, NPTH, F.Cu at (165.7, 61.1)
- added REF**: NPTH, NPTH, F.Cu at (120.6, 71.8)
- added REF**: NPTH, NPTH, F.Cu at (104.4, 106.2)
- added REF**: NPTH, NPTH, F.Cu at (184.5, 97.1)
- added REF**: NPTH, NPTH, F.Cu at (167.3, 44.9)
- added REF**: NPTH, NPTH, F.Cu at (185.3, 97.1)
- added REF**: NPTH, NPTH, F.Cu at (104.4, 107.8)
- added REF**: NPTH, NPTH, F.Cu at (111.7, 44.9)
- added REF**: NPTH, NPTH, F.Cu at (184.5, 98.9)
- added REF**: NPTH, NPTH, F.Cu at (174.6, 71.0)
- added REF**: NPTH, NPTH, F.Cu at (185.3, 98.9)
- added REF**: NPTH, NPTH, F.Cu at (111.7, 61.1)
- added REF**: NPTH, NPTH, F.Cu at (158.4, 89.0)
- added REF**: NPTH, NPTH, F.Cu at (122.4, 34.2)
- added REF**: NPTH, NPTH, F.Cu at (104.4, 53.8)
- added REF**: NPTH, NPTH, F.Cu at (156.6, 71.0)
- added REF**: NPTH, NPTH, F.Cu at (167.3, 61.1)
- added REF**: NPTH, NPTH, F.Cu at (174.6, 34.2)
- added REF**: NPTH, NPTH, F.Cu at (130.5, 44.9)
- added REF**: NPTH, NPTH, F.Cu at (104.4, 52.2)
- added REF**: NPTH, NPTH, F.Cu at (140.4, 106.2)
- added REF**: NPTH, NPTH, F.Cu at (140.4, 53.8)
- added REF**: NPTH, NPTH, F.Cu at (140.4, 107.8)
- added REF**: NPTH, NPTH, F.Cu at (131.3, 61.1)
- added REF**: NPTH, NPTH, F.Cu at (130.5, 62.9)
- added REF**: NPTH, NPTH, F.Cu at (113.3, 26.9)
- added REF**: NPTH, NPTH, F.Cu at (166.5, 98.9)
- added REF**: NPTH, NPTH, F.Cu at (176.4, 53.8)
- added REF**: NPTH, NPTH, F.Cu at (184.5, 115.1)
- added REF**: NPTH, NPTH, F.Cu at (174.6, 107.8)
- added REF**: NPTH, NPTH, F.Cu at (176.4, 70.2)
- added REF**: NPTH, NPTH, F.Cu at (192.6, 107.0)
- added REF**: NPTH, NPTH, F.Cu at (138.6, 71.0)
- added REF**: NPTH, NPTH, F.Cu at (158.4, 107.0)
- added REF**: NPTH, NPTH, F.Cu at (113.3, 80.9)
- added REF**: NPTH, NPTH, F.Cu at (166.5, 26.9)
- added REF**: NPTH, NPTH, F.Cu at (185.3, 80.9)
- added REF**: NPTH, NPTH, F.Cu at (156.6, 89.8)
- added REF**: NPTH, NPTH, F.Cu at (176.4, 107.8)
- added REF**: NPTH, NPTH, F.Cu at (174.6, 35.0)
- added REF**: NPTH, NPTH, F.Cu at (156.6, 35.8)
- added REF**: NPTH, NPTH, F.Cu at (111.7, 115.1)
- added REF**: NPTH, NPTH, F.Cu at (158.4, 89.8)
- added REF**: NPTH, NPTH, F.Cu at (148.5, 62.9)
- added REF**: NPTH, NPTH, F.Cu at (183.7, 62.9)
- added REF**: NPTH, NPTH, F.Cu at (147.7, 98.9)
- added REF**: NPTH, NPTH, F.Cu at (192.6, 89.8)
- added REF**: NPTH, NPTH, F.Cu at (184.5, 61.1)
- added REF**: NPTH, NPTH, F.Cu at (111.7, 62.9)
- added REF**: NPTH, NPTH, F.Cu at (131.3, 44.9)
- added REF**: NPTH, NPTH, F.Cu at (167.3, 79.1)
- added REF**: NPTH, NPTH, F.Cu at (156.6, 106.2)
- added REF**: NPTH, NPTH, F.Cu at (183.7, 97.1)
- added REF**: NPTH, NPTH, F.Cu at (122.4, 53.0)
- added REF**: NPTH, NPTH, F.Cu at (185.3, 62.9)
- added REF**: NPTH, NPTH, F.Cu at (131.3, 97.1)
- added REF**: NPTH, NPTH, F.Cu at (112.5, 43.1)
- added REF**: NPTH, NPTH, F.Cu at (129.7, 62.9)
- added REF**: NPTH, NPTH, F.Cu at (147.7, 26.9)
- added REF**: NPTH, NPTH, F.Cu at (158.4, 88.2)
- added REF**: NPTH, NPTH, F.Cu at (183.7, 61.1)
- added REF**: NPTH, NPTH, F.Cu at (122.4, 89.0)
- added REF**: NPTH, NPTH, F.Cu at (129.7, 44.9)
- added REF**: NPTH, NPTH, F.Cu at (192.6, 70.2)
- added REF**: NPTH, NPTH, F.Cu at (174.6, 35.8)
- added REF**: NPTH, NPTH, F.Cu at (165.7, 80.9)
- added REF**: NPTH, NPTH, F.Cu at (140.4, 71.8)
- added REF**: NPTH, NPTH, F.Cu at (129.7, 26.9)
- added REF**: NPTH, NPTH, F.Cu at (158.4, 71.0)
- added REF**: NPTH, NPTH, F.Cu at (176.4, 88.2)
- added REF**: NPTH, NPTH, F.Cu at (192.6, 89.0)
- added REF**: NPTH, NPTH, F.Cu at (158.4, 53.0)
- added REF**: NPTH, NPTH, F.Cu at (156.6, 70.2)
- added REF**: NPTH, NPTH, F.Cu at (138.6, 71.8)
- added REF**: NPTH, NPTH, F.Cu at (147.7, 115.1)
- added REF**: NPTH, NPTH, F.Cu at (149.3, 79.1)
- added REF**: NPTH, NPTH, F.Cu at (176.4, 71.0)
- added REF**: NPTH, NPTH, F.Cu at (140.4, 53.0)
- added REF**: NPTH, NPTH, F.Cu at (140.4, 52.2)
- added REF**: NPTH, NPTH, F.Cu at (130.5, 26.9)
- added REF**: NPTH, NPTH, F.Cu at (120.6, 71.0)
- added REF**: NPTH, NPTH, F.Cu at (138.6, 35.0)
- added REF**: NPTH, NPTH, F.Cu at (176.4, 89.0)
- added REF**: NPTH, NPTH, F.Cu at (165.7, 26.9)
- added REF**: NPTH, NPTH, F.Cu at (122.4, 53.8)
- added REF**: NPTH, NPTH, F.Cu at (148.5, 43.1)
- added REF**: NPTH, NPTH, F.Cu at (122.4, 71.0)
- added REF**: NPTH, NPTH, F.Cu at (112.5, 97.1)
- added REF**: NPTH, NPTH, F.Cu at (149.3, 97.1)
- added REF**: NPTH, NPTH, F.Cu at (138.6, 107.8)
- added REF**: NPTH, NPTH, F.Cu at (130.5, 80.9)
- added REF**: NPTH, NPTH, F.Cu at (130.5, 61.1)
- added REF**: NPTH, NPTH, F.Cu at (192.6, 107.8)
- added REF**: NPTH, NPTH, F.Cu at (120.6, 107.8)
- added REF**: NPTH, NPTH, F.Cu at (120.6, 53.8)
- added REF**: NPTH, NPTH, F.Cu at (122.4, 88.2)
- added REF**: NPTH, NPTH, F.Cu at (120.6, 35.8)
- added REF**: NPTH, NPTH, F.Cu at (167.3, 80.9)
- added REF**: NPTH, NPTH, F.Cu at (165.7, 43.1)
- added REF**: NPTH, NPTH, F.Cu at (112.5, 26.9)
- added REF**: NPTH, NPTH, F.Cu at (138.6, 107.0)
- added REF**: NPTH, NPTH, F.Cu at (149.3, 98.9)
- added REF**: NPTH, NPTH, F.Cu at (183.7, 26.9)
- added REF**: NPTH, NPTH, F.Cu at (156.6, 34.2)
- added REF**: NPTH, NPTH, F.Cu at (113.3, 97.1)
- added REF**: NPTH, NPTH, F.Cu at (120.6, 89.0)
- added REF**: NPTH, NPTH, F.Cu at (184.5, 44.9)
- added REF**: NPTH, NPTH, F.Cu at (185.3, 26.9)
- added REF**: NPTH, NPTH, F.Cu at (122.4, 35.0)
- added REF**: NPTH, NPTH, F.Cu at (113.3, 79.1)
- added REF**: NPTH, NPTH, F.Cu at (104.4, 35.8)
- added REF**: NPTH, NPTH, F.Cu at (174.6, 53.0)
- added REF**: NPTH, NPTH, F.Cu at (167.3, 62.9)
- added REF**: NPTH, NPTH, F.Cu at (148.5, 44.9)
- added REF**: NPTH, NPTH, F.Cu at (166.5, 44.9)
- added REF**: NPTH, NPTH, F.Cu at (149.3, 44.9)
- added REF**: NPTH, NPTH, F.Cu at (131.3, 79.1)
- added REF**: NPTH, NPTH, F.Cu at (192.6, 35.0)
- added REF**: NPTH, NPTH, F.Cu at (183.7, 80.9)
- added REF**: NPTH, NPTH, F.Cu at (176.4, 34.2)
- added REF**: NPTH, NPTH, F.Cu at (176.4, 53.0)
- added REF**: NPTH, NPTH, F.Cu at (147.7, 97.1)
- added REF**: NPTH, NPTH, F.Cu at (156.6, 71.8)
- added REF**: NPTH, NPTH, F.Cu at (112.5, 44.9)
- added REF**: NPTH, NPTH, F.Cu at (129.7, 43.1)
- added REF**: NPTH, NPTH, F.Cu at (120.6, 89.8)
- added REF**: NPTH, NPTH, F.Cu at (183.7, 79.1)
- added REF**: NPTH, NPTH, F.Cu at (158.4, 53.8)
- added REF**: NPTH, NPTH, F.Cu at (149.3, 80.9)
- added REF**: NPTH, NPTH, F.Cu at (120.6, 107.0)
- added REF**: NPTH, NPTH, F.Cu at (138.6, 34.2)
- added REF**: NPTH, NPTH, F.Cu at (111.7, 97.1)
- added REF**: NPTH, NPTH, F.Cu at (174.6, 70.2)
- added REF**: NPTH, NPTH, F.Cu at (185.3, 43.1)
- added REF**: NPTH, NPTH, F.Cu at (185.3, 79.1)
- added REF**: NPTH, NPTH, F.Cu at (104.4, 89.0)
- added REF**: NPTH, NPTH, F.Cu at (158.4, 52.2)
- added REF**: NPTH, NPTH, F.Cu at (156.6, 53.8)
- added REF**: Fiducial, Fiducial, F.Cu at (100.0, 119.5)
- added REF**: NPTH, NPTH, F.Cu at (184.5, 79.1)
- added REF**: NPTH, NPTH, F.Cu at (120.6, 106.2)
- added REF**: NPTH, NPTH, F.Cu at (165.7, 98.9)
- added REF**: NPTH, NPTH, F.Cu at (158.4, 107.8)
- added REF**: NPTH, NPTH, F.Cu at (129.7, 97.1)
- added REF**: NPTH, NPTH, F.Cu at (156.6, 107.0)
- added REF**: NPTH, NPTH, F.Cu at (130.5, 98.9)
- added REF**: NPTH, NPTH, F.Cu at (167.3, 26.9)
- added REF**: NPTH, NPTH, F.Cu at (140.4, 35.0)
- added REF**: NPTH, NPTH, F.Cu at (148.5, 97.1)
- added REF**: NPTH, NPTH, F.Cu at (104.4, 88.2)
- added REF**: NPTH, NPTH, F.Cu at (165.7, 62.9)
- added REF**: NPTH, NPTH, F.Cu at (112.5, 98.9)
- added REF**: NPTH, NPTH, F.Cu at (111.7, 79.1)
- added REF**: NPTH, NPTH, F.Cu at (147.7, 80.9)
- added REF**: NPTH, NPTH, F.Cu at (140.4, 34.2)
- added REF**: NPTH, NPTH, F.Cu at (113.3, 115.1)
- added REF**: NPTH, NPTH, F.Cu at (140.4, 89.8)
- added REF**: NPTH, NPTH, F.Cu at (138.6, 89.0)
- added REF**: NPTH, NPTH, F.Cu at (167.3, 98.9)
- added REF**: NPTH, NPTH, F.Cu at (131.3, 80.9)
- added REF**: NPTH, NPTH, F.Cu at (184.5, 80.9)
- added REF**: NPTH, NPTH, F.Cu at (104.4, 70.2)
- added REF**: NPTH, NPTH, F.Cu at (185.3, 61.1)
- added REF**: NPTH, NPTH, F.Cu at (166.5, 97.1)
- added REF**: NPTH, NPTH, F.Cu at (122.4, 107.0)
- added REF**: NPTH, NPTH, F.Cu at (112.5, 80.9)
- added REF**: NPTH, NPTH, F.Cu at (167.3, 115.1)
- added REF**: NPTH, NPTH, F.Cu at (176.4, 89.8)
- added REF**: NPTH, NPTH, F.Cu at (176.4, 106.2)
- added REF**: NPTH, NPTH, F.Cu at (147.7, 61.1)
- added REF**: NPTH, NPTH, F.Cu at (174.6, 71.8)
- added REF**: NPTH, NPTH, F.Cu at (140.4, 71.0)
- added REF**: NPTH, NPTH, F.Cu at (183.7, 43.1)
- added REF**: NPTH, NPTH, F.Cu at (131.3, 26.9)
- added REF**: NPTH, NPTH, F.Cu at (138.6, 70.2)
- added REF**: NPTH, NPTH, F.Cu at (149.3, 62.9)
- added REF**: NPTH, NPTH, F.Cu at (174.6, 53.8)
- added REF**: NPTH, NPTH, F.Cu at (129.7, 61.1)
- added REF**: NPTH, NPTH, F.Cu at (129.7, 98.9)
- added REF**: NPTH, NPTH, F.Cu at (167.3, 97.1)
- added REF**: NPTH, NPTH, F.Cu at (140.4, 70.2)
- added REF**: NPTH, NPTH, F.Cu at (149.3, 43.1)
- added REF**: NPTH, NPTH, F.Cu at (120.6, 35.0)
- added REF**: NPTH, NPTH, F.Cu at (148.5, 115.1)
- added REF**: Fiducial, Fiducial, B.Cu at (100.0, 119.5)
- added REF**: Fiducial, Fiducial, B.Cu at (197.0, 22.5)
- added REF**: Fiducial, Fiducial, B.Cu at (100.0, 22.5)
- added REF**: NPTH, NPTH, F.Cu at (185.3, 44.9)
- added REF**: NPTH, NPTH, F.Cu at (111.7, 98.9)
- added REF**: NPTH, NPTH, F.Cu at (131.3, 98.9)
- added REF**: NPTH, NPTH, F.Cu at (183.7, 115.1)
- added REF**: NPTH, NPTH, F.Cu at (192.6, 53.0)
- added REF**: NPTH, NPTH, F.Cu at (165.7, 115.1)
- added REF**: NPTH, NPTH, F.Cu at (176.4, 52.2)
- added REF**: NPTH, NPTH, F.Cu at (104.4, 71.0)
- added REF**: NPTH, NPTH, F.Cu at (192.6, 34.2)
- added REF**: NPTH, NPTH, F.Cu at (192.6, 71.8)
- added REF**: NPTH, NPTH, F.Cu at (192.6, 52.2)
- added REF**: NPTH, NPTH, F.Cu at (138.6, 106.2)
- added REF**: NPTH, NPTH, F.Cu at (149.3, 115.1)
- added REF**: NPTH, NPTH, F.Cu at (156.6, 52.2)
- added REF**: NPTH, NPTH, F.Cu at (149.3, 61.1)
- added REF**: NPTH, NPTH, F.Cu at (113.3, 62.9)
- added REF**: NPTH, NPTH, F.Cu at (148.5, 98.9)
- added REF**: NPTH, NPTH, F.Cu at (120.6, 70.2)
- added REF**: NPTH, NPTH, F.Cu at (122.4, 70.2)
- added REF**: NPTH, NPTH, F.Cu at (138.6, 53.8)
- added REF**: NPTH, NPTH, F.Cu at (112.5, 79.1)
- added REF**: NPTH, NPTH, F.Cu at (104.4, 107.0)
- added REF**: NPTH, NPTH, F.Cu at (158.4, 106.2)
- added REF**: NPTH, NPTH, F.Cu at (148.5, 61.1)
- added REF**: NPTH, NPTH, F.Cu at (165.7, 97.1)
- added REF**: NPTH, NPTH, F.Cu at (112.5, 61.1)
- added REF**: NPTH, NPTH, F.Cu at (113.3, 61.1)
- added REF**: NPTH, NPTH, F.Cu at (111.7, 43.1)
- added REF**: NPTH, NPTH, F.Cu at (147.7, 44.9)
- added REF**: NPTH, NPTH, F.Cu at (113.3, 44.9)
- added REF**: NPTH, NPTH, F.Cu at (192.6, 35.8)
- added REF**: NPTH, NPTH, F.Cu at (156.6, 89.0)
- added REF**: NPTH, NPTH, F.Cu at (147.7, 43.1)
- added REF**: NPTH, NPTH, F.Cu at (122.4, 107.8)
- added REF**: NPTH, NPTH, F.Cu at (174.6, 107.0)
- added REF**: NPTH, NPTH, F.Cu at (138.6, 52.2)
- added REF**: NPTH, NPTH, F.Cu at (174.6, 89.8)
- added REF**: NPTH, NPTH, F.Cu at (174.6, 89.0)
- added REF**: NPTH, NPTH, F.Cu at (174.6, 88.2)
- added REF**: NPTH, NPTH, F.Cu at (166.5, 115.1)
- added REF**: NPTH, NPTH, F.Cu at (122.4, 52.2)
- added REF**: NPTH, NPTH, F.Cu at (130.5, 115.1)
- added REF**: NPTH, NPTH, F.Cu at (166.5, 62.9)
- added REF**: NPTH, NPTH, F.Cu at (120.6, 34.2)
- added REF**: NPTH, NPTH, F.Cu at (111.7, 26.9)
- added REF**: NPTH, NPTH, F.Cu at (184.5, 26.9)
- added REF**: Fiducial, Fiducial, F.Cu at (100.0, 22.5)
- added REF**: NPTH, NPTH, F.Cu at (183.7, 98.9)
- added REF**: NPTH, NPTH, F.Cu at (156.6, 107.8)
- added REF**: NPTH, NPTH, F.Cu at (104.4, 71.8)
- added REF**: NPTH, NPTH, F.Cu at (120.6, 53.0)
- added REF**: NPTH, NPTH, F.Cu at (156.6, 53.0)
- added REF**: NPTH, NPTH, F.Cu at (183.7, 44.9)
- added REF**: NPTH, NPTH, F.Cu at (158.4, 71.8)
- added REF**: NPTH, NPTH, F.Cu at (185.3, 115.1)
- added REF**: NPTH, NPTH, F.Cu at (131.3, 62.9)
- added REF**: NPTH, NPTH, F.Cu at (192.6, 71.0)
- added REF**: NPTH, NPTH, F.Cu at (166.5, 79.1)
- added REF**: NPTH, NPTH, F.Cu at (122.4, 71.8)
- added REF**: NPTH, NPTH, F.Cu at (122.4, 89.8)
- added REF**: NPTH, NPTH, F.Cu at (166.5, 61.1)
Other:
- outline, holes or cut-outs redrawn

Commit message: panels
Parts:
- removed the REF** at (197.0, 22.5) (x2)
- removed the REF** at (100.0, 119.5) (x2)
- removed the REF** at (100.0, 22.5) (x2)
- added REF**: Fiducial, Fiducial, F.Cu at (100.0, 22.5)
- added REF**: Fiducial, Fiducial, F.Cu at (197.0, 22.5)
- added REF**: Fiducial, Fiducial, F.Cu at (100.0, 119.5)
- added REF**: Fiducial, Fiducial, B.Cu at (100.0, 119.5)
- added REF**: Fiducial, Fiducial, B.Cu at (100.0, 22.5)
- added REF**: Fiducial, Fiducial, B.Cu at (197.0, 22.5)

Commit message: gerbers
Parts:
- removed the REF** at (158.4, 88.2)
- removed the REF** at (113.3, 98.9)
- removed the REF** at (130.5, 115.1)
- removed the REF** at (122.4, 89.0)
- removed the REF** at (140.4, 35.0)
- removed the REF** at (104.4, 70.2)
- removed the REF** at (138.6, 89.8)
- removed the REF** at (112.5, 115.1)
- removed the REF** at (111.7, 44.9)
- removed the REF** at (120.6, 107.8)
- removed the REF** at (129.7, 62.9)
- removed the REF** at (104.4, 53.0)
- removed the REF** at (158.4, 52.2)
- removed the REF** at (149.3, 62.9)
- removed the REF** at (104.4, 53.8)
- removed the REF** at (138.6, 52.2)
- removed the REF** at (140.4, 35.8)
- removed the REF** at (120.6, 106.2)
- removed the REF** at (122.4, 89.8)
- removed the REF** at (167.3, 79.1)
- removed the REF** at (158.4, 89.0)
- removed the REF** at (183.7, 26.9)
- removed the REF** at (120.6, 71.0)
- removed the REF** at (176.4, 106.2)
- removed the REF** at (122.4, 107.8)
- removed the REF** at (104.4, 88.2)
- removed the REF** at (131.3, 97.1)
- removed the REF** at (149.3, 26.9)
- removed the REF** at (156.6, 70.2)
- removed the REF** at (130.5, 44.9)
- removed the REF** at (112.5, 26.9)
- removed the REF** at (149.3, 98.9)
- removed the REF** at (129.7, 44.9)
- removed the REF** at (184.5, 79.1)
- removed the REF** at (131.3, 98.9)
- removed the REF** at (174.6, 53.0)
- removed the REF** at (113.3, 97.1)
- removed the REF** at (120.6, 53.0)
- removed the REF** at (122.4, 71.8)
- removed the REF** at (149.3, 115.1)
- removed the REF** at (129.7, 61.1)
- removed the REF** at (113.3, 115.1)
- removed the REF** at (174.6, 107.0)
- removed the REF** at (113.3, 44.9)
- removed the REF** at (156.6, 107.8)
- removed the REF** at (131.3, 61.1)
- removed the REF** at (183.7, 80.9)
- removed the REF** at (140.4, 89.0)
- removed the REF** at (183.7, 115.1)
- removed the REF** at (100.0, 22.5) (x2)
- removed the REF** at (166.5, 62.9)
- removed the REF** at (140.4, 70.2)
- removed the REF** at (176.4, 52.2)
- removed the REF** at (140.4, 88.2)
- removed the REF** at (112.5, 97.1)
- removed the REF** at (148.5, 44.9)
- removed the REF** at (166.5, 80.9)
- removed the REF** at (174.6, 89.0)
- removed the REF** at (156.6, 53.0)
- removed the REF** at (192.6, 70.2)
- removed the REF** at (176.4, 35.8)
- removed the REF** at (192.6, 53.0)
- removed the REF** at (183.7, 43.1)
- removed the REF** at (158.4, 89.8)
- removed the REF** at (174.6, 89.8)
- removed the REF** at (113.3, 61.1)
- removed the REF** at (129.7, 97.1)
- removed the REF** at (113.3, 79.1)
- removed the REF** at (167.3, 44.9)
- removed the REF** at (165.7, 115.1)
- removed the REF** at (166.5, 97.1)
- removed the REF** at (185.3, 62.9)
- removed the REF** at (165.7, 44.9)
- removed the REF** at (138.6, 35.8)
- removed the REF** at (185.3, 79.1)
- removed the REF** at (104.4, 107.0)
- removed the REF** at (192.6, 107.8)
- removed the REF** at (174.6, 53.8)
- removed the REF** at (165.7, 80.9)
- removed the REF** at (147.7, 97.1)
- removed the REF** at (148.5, 61.1)
- removed the REF** at (140.4, 89.8)
- removed the REF** at (156.6, 52.2)
- removed the REF** at (122.4, 52.2)
- removed the REF** at (185.3, 43.1)
- removed the REF** at (192.6, 71.8)
- removed the REF** at (192.6, 107.0)
- removed the REF** at (148.5, 62.9)
- removed the REF** at (122.4, 71.0)
- removed the REF** at (167.3, 97.1)
- removed the REF** at (165.7, 26.9)
- removed the REF** at (130.5, 62.9)
- removed the REF** at (156.6, 53.8)
- removed the REF** at (148.5, 26.9)
- removed the REF** at (158.4, 71.8)
- removed the REF** at (111.7, 43.1)
- removed the REF** at (158.4, 35.0)
- removed the REF** at (148.5, 98.9)
- removed the REF** at (167.3, 115.1)
- removed the REF** at (184.5, 43.1)
- removed the REF** at (184.5, 115.1)
- removed the REF** at (104.4, 34.2)
- removed the REF** at (148.5, 79.1)
- removed the REF** at (147.7, 79.1)
- removed the REF** at (197.0, 22.5) (x2)
- removed the REF** at (131.3, 44.9)
- removed the REF** at (176.4, 53.0)
- removed the REF** at (129.7, 80.9)
- removed the REF** at (138.6, 107.0)
- removed the REF** at (183.7, 44.9)
- removed the REF** at (112.5, 61.1)
- removed the REF** at (100.0, 119.5) (x2)
- removed the REF** at (138.6, 53.8)
- removed the REF** at (149.3, 44.9)
- removed the REF** at (176.4, 53.8)
- removed the REF** at (192.6, 71.0)
- removed the REF** at (156.6, 107.0)
- removed the REF** at (156.6, 89.8)
- removed the REF** at (138.6, 35.0)
- removed the REF** at (111.7, 26.9)
- removed the REF** at (174.6, 70.2)
- removed the REF** at (131.3, 43.1)
- removed the REF** at (129.7, 26.9)
- removed the REF** at (176.4, 89.0)
- removed the REF** at (140.4, 71.0)
- removed the REF** at (104.4, 107.8)
- removed the REF** at (176.4, 107.8)
- removed the REF** at (112.5, 62.9)
- removed the REF** at (112.5, 44.9)
- removed the REF** at (112.5, 98.9)
- removed the REF** at (122.4, 70.2)
- removed the REF** at (185.3, 97.1)
- removed the REF** at (176.4, 107.0)
- removed the REF** at (156.6, 71.8)
- removed the REF** at (113.3, 80.9)
- removed the REF** at (131.3, 80.9)
- removed the REF** at (104.4, 106.2)
- removed the REF** at (104.4, 89.0)
- removed the REF** at (174.6, 52.2)
- removed the REF** at (184.5, 44.9)
- removed the REF** at (129.7, 43.1)
- removed the REF** at (140.4, 71.8)
- removed the REF** at (111.7, 62.9)
- removed the REF** at (147.7, 62.9)
- removed the REF** at (184.5, 98.9)
- removed the REF** at (174.6, 71.0)
- removed the REF** at (174.6, 71.8)
- removed the REF** at (122.4, 53.0)
- removed the REF** at (185.3, 44.9)
- removed the REF** at (147.7, 61.1)
- removed the REF** at (111.7, 98.9)
- removed the REF** at (185.3, 80.9)
- removed the REF** at (122.4, 88.2)
- removed the REF** at (120.6, 89.8)
- removed the REF** at (192.6, 89.0)
- removed the REF** at (131.3, 79.1)
- removed the REF** at (112.5, 43.1)
- removed the REF** at (138.6, 89.0)
- removed the REF** at (148.5, 43.1)
- removed the REF** at (147.7, 115.1)
- removed the REF** at (140.4, 106.2)
- removed the REF** at (120.6, 70.2)
- removed the REF** at (138.6, 106.2)
- removed the REF** at (138.6, 88.2)
- removed the REF** at (167.3, 62.9)
- removed the REF** at (156.6, 35.8)
- removed the REF** at (131.3, 115.1)
- removed the REF** at (138.6, 70.2)
- removed the REF** at (183.7, 79.1)
- removed the REF** at (185.3, 26.9)
- removed the REF** at (166.5, 115.1)
- removed the REF** at (158.4, 35.8)
- removed the REF** at (113.3, 62.9)
- removed the REF** at (158.4, 70.2)
- removed the REF** at (131.3, 62.9)
- removed the REF** at (167.3, 98.9)
- removed the REF** at (165.7, 98.9)
- removed the REF** at (183.7, 62.9)
- removed the REF** at (129.7, 98.9)
- removed the REF** at (111.7, 79.1)
- removed the REF** at (120.6, 71.8)
- removed the REF** at (185.3, 115.1)
- removed the REF** at (184.5, 61.1)
- removed the REF** at (130.5, 61.1)
- removed the REF** at (149.3, 97.1)
- removed the REF** at (122.4, 53.8)
- removed the REF** at (156.6, 71.0)
- removed the REF** at (122.4, 34.2)
- removed the REF** at (174.6, 88.2)
- removed the REF** at (140.4, 107.0)
- removed the REF** at (130.5, 79.1)
- removed the REF** at (158.4, 71.0)
- removed the REF** at (140.4, 52.2)
- removed the REF** at (167.3, 26.9)
- removed the REF** at (122.4, 107.0)
- removed the REF** at (148.5, 115.1)
- removed the REF** at (147.7, 98.9)
- removed the REF** at (183.7, 98.9)
- removed the REF** at (176.4, 70.2)
- removed the REF** at (147.7, 44.9)
- removed the REF** at (165.7, 61.1)
- removed the REF** at (192.6, 88.2)
- removed the REF** at (149.3, 80.9)
- removed the REF** at (129.7, 79.1)
- removed the REF** at (138.6, 34.2)
- removed the REF** at (140.4, 53.0)
- removed the REF** at (165.7, 97.1)
- removed the REF** at (138.6, 107.8)
- removed the REF** at (120.6, 107.0)
- removed the REF** at (149.3, 61.1)
- removed the REF** at (149.3, 43.1)
- removed the REF** at (131.3, 26.9)
- removed the REF** at (112.5, 79.1)
- removed the REF** at (176.4, 89.8)
- removed the REF** at (138.6, 53.0)
- removed the REF** at (147.7, 26.9)
- removed the REF** at (158.4, 107.8)
- removed the REF** at (138.6, 71.0)
- removed the REF** at (104.4, 52.2)
- removed the REF** at (176.4, 34.2)
- removed the REF** at (130.5, 26.9)
- removed the REF** at (158.4, 53.8)
- removed the REF** at (158.4, 34.2)
- removed the REF** at (166.5, 44.9)
- removed the REF** at (166.5, 26.9)
- removed the REF** at (140.4, 53.8)
- removed the REF** at (156.6, 106.2)
- removed the REF** at (104.4, 71.0)
- removed the REF** at (192.6, 34.2)
- removed the REF** at (120.6, 35.0)
- removed the REF** at (122.4, 35.8)
- removed the REF** at (104.4, 71.8)
- removed the REF** at (147.7, 43.1)
- removed the REF** at (130.5, 97.1)
- removed the REF** at (184.5, 80.9)
- removed the REF** at (120.6, 34.2)
- removed the REF** at (184.5, 62.9)
- removed the REF** at (167.3, 43.1)
- removed the REF** at (120.6, 35.8)
- removed the REF** at (120.6, 52.2)
- removed the REF** at (192.6, 89.8)
- removed the REF** at (156.6, 34.2)
- removed the REF** at (192.6, 35.0)
- removed the REF** at (140.4, 107.8)
- removed the REF** at (174.6, 35.0)
- removed the REF** at (158.4, 107.0)
- removed the REF** at (111.7, 80.9)
- removed the REF** at (166.5, 43.1)
- removed the REF** at (147.7, 80.9)
- removed the REF** at (176.4, 71.8)
- removed the REF** at (104.4, 89.8)
- removed the REF** at (192.6, 53.8)
- removed the REF** at (130.5, 98.9)
- removed the REF** at (174.6, 34.2)
- removed the REF** at (174.6, 106.2)
- removed the REF** at (167.3, 80.9)
- removed the REF** at (156.6, 89.0)
- removed the REF** at (165.7, 79.1)
- removed the REF** at (192.6, 52.2)
- removed the REF** at (185.3, 61.1)
- removed the REF** at (122.4, 106.2)
- removed the REF** at (183.7, 61.1)
- removed the REF** at (176.4, 71.0)
- removed the REF** at (113.3, 26.9)
- removed the REF** at (111.7, 115.1)
- removed the REF** at (174.6, 35.8)
- removed the REF** at (166.5, 98.9)
- removed the REF** at (113.3, 43.1)
- removed the REF** at (167.3, 61.1)
- removed the REF** at (140.4, 34.2)
- removed the REF** at (120.6, 53.8)
- removed the REF** at (130.5, 80.9)
- removed the REF** at (104.4, 35.8)
- removed the REF** at (122.4, 35.0)
- removed the REF** at (165.7, 62.9)
- removed the REF** at (158.4, 106.2)
- removed the REF** at (112.5, 80.9)
- removed the REF** at (148.5, 97.1)
- removed the REF** at (138.6, 71.8)
- removed the REF** at (184.5, 26.9)
- removed the REF** at (104.4, 35.0)
- removed the REF** at (148.5, 80.9)
- removed the REF** at (192.6, 35.8)
- removed the REF** at (111.7, 61.1)
- removed the REF** at (120.6, 88.2)
- removed the REF** at (165.7, 43.1)
- removed the REF** at (156.6, 88.2)
- removed the REF** at (174.6, 107.8)
- removed the REF** at (166.5, 61.1)
- removed the REF** at (149.3, 79.1)
- removed the REF** at (111.7, 97.1)
- removed the REF** at (176.4, 35.0)
- removed the REF** at (166.5, 79.1)
- removed the REF** at (130.5, 43.1)
- removed the REF** at (176.4, 88.2)
- removed the REF** at (184.5, 97.1)
- removed the REF** at (192.6, 106.2)
- removed the REF** at (129.7, 115.1)
- removed the REF** at (120.6, 89.0)
- removed the REF** at (183.7, 97.1)
- removed the REF** at (156.6, 35.0)
- removed the REF** at (158.4, 53.0)
- removed the REF** at (185.3, 98.9)
- added REF**: NPTH, NPTH, F.Cu at (184.9, 44.9)
- added REF**: NPTH, NPTH, F.Cu at (112.9, 62.9)
- added REF**: NPTH, NPTH, F.Cu at (184.9, 26.9)
- added REF**: NPTH, NPTH, F.Cu at (192.6, 89.4)
- added REF**: NPTH, NPTH, F.Cu at (112.1, 97.1)
- added REF**: NPTH, NPTH, F.Cu at (166.9, 98.9)
- added REF**: NPTH, NPTH, F.Cu at (148.1, 115.1)
- added REF**: NPTH, NPTH, F.Cu at (112.1, 61.1)
- added REF**: NPTH, NPTH, F.Cu at (174.6, 88.6)
- added REF**: NPTH, NPTH, F.Cu at (184.9, 98.9)
- added REF**: NPTH, NPTH, F.Cu at (122.4, 53.4)
- added REF**: NPTH, NPTH, F.Cu at (156.6, 107.4)
- added REF**: NPTH, NPTH, F.Cu at (122.4, 88.6)
- added REF**: NPTH, NPTH, F.Cu at (158.4, 34.6)
- added REF**: NPTH, NPTH, F.Cu at (166.9, 79.1)
- added REF**: NPTH, NPTH, F.Cu at (174.6, 71.4)
- added REF**: NPTH, NPTH, F.Cu at (166.1, 79.1)
- added REF**: NPTH, NPTH, F.Cu at (112.9, 61.1)
- added REF**: NPTH, NPTH, F.Cu at (158.4, 53.4)
- added REF**: NPTH, NPTH, F.Cu at (184.9, 97.1)
- added REF**: NPTH, NPTH, F.Cu at (122.4, 71.4)
- added REF**: NPTH, NPTH, F.Cu at (130.1, 97.1)
- added REF**: NPTH, NPTH, F.Cu at (104.4, 34.6)
- added REF**: NPTH, NPTH, F.Cu at (148.1, 62.9)
- added REF**: NPTH, NPTH, F.Cu at (148.9, 61.1)
- added REF**: NPTH, NPTH, F.Cu at (166.1, 61.1)
- added REF**: NPTH, NPTH, F.Cu at (112.1, 62.9)
- added REF**: NPTH, NPTH, F.Cu at (140.4, 89.4)
- added REF**: NPTH, NPTH, F.Cu at (156.6, 71.4)
- added REF**: Fiducial, Fiducial, F.Cu at (100.0, 119.5)
- added REF**: NPTH, NPTH, F.Cu at (130.9, 43.1)
- added REF**: NPTH, NPTH, F.Cu at (176.4, 107.4)
- added REF**: NPTH, NPTH, F.Cu at (130.9, 62.9)
- added REF**: NPTH, NPTH, F.Cu at (184.1, 98.9)
- added REF**: NPTH, NPTH, F.Cu at (148.9, 26.9)
- added REF**: NPTH, NPTH, F.Cu at (174.6, 106.6)
- added REF**: NPTH, NPTH, F.Cu at (174.6, 70.6)
- added REF**: NPTH, NPTH, F.Cu at (120.6, 107.4)
- added REF**: NPTH, NPTH, F.Cu at (148.1, 43.1)
- added REF**: NPTH, NPTH, F.Cu at (148.1, 26.9)
- added REF**: NPTH, NPTH, F.Cu at (130.1, 26.9)
- added REF**: NPTH, NPTH, F.Cu at (120.6, 52.6)
- added REF**: NPTH, NPTH, F.Cu at (166.1, 80.9)
- added REF**: NPTH, NPTH, F.Cu at (166.9, 80.9)
- added REF**: NPTH, NPTH, F.Cu at (104.4, 52.6)
- added REF**: NPTH, NPTH, F.Cu at (166.1, 97.1)
- added REF**: NPTH, NPTH, F.Cu at (120.6, 71.4)
- added REF**: NPTH, NPTH, F.Cu at (130.9, 97.1)
- added REF**: NPTH, NPTH, F.Cu at (148.9, 79.1)
- added REF**: NPTH, NPTH, F.Cu at (130.9, 61.1)
- added REF**: NPTH, NPTH, F.Cu at (130.9, 98.9)
- added REF**: NPTH, NPTH, F.Cu at (130.1, 79.1)
- added REF**: NPTH, NPTH, F.Cu at (104.4, 88.6)
- added REF**: NPTH, NPTH, F.Cu at (148.9, 97.1)
- added REF**: NPTH, NPTH, F.Cu at (140.4, 71.4)
- added REF**: NPTH, NPTH, F.Cu at (156.6, 35.4)
- added REF**: NPTH, NPTH, F.Cu at (184.1, 43.1)
- added REF**: NPTH, NPTH, F.Cu at (122.4, 35.4)
- added REF**: NPTH, NPTH, F.Cu at (176.4, 88.6)
- added REF**: NPTH, NPTH, F.Cu at (104.4, 53.4)
- added REF**: NPTH, NPTH, F.Cu at (174.6, 52.6)
- added REF**: NPTH, NPTH, F.Cu at (192.6, 107.4)
- added REF**: NPTH, NPTH, F.Cu at (184.1, 115.1)
- added REF**: NPTH, NPTH, F.Cu at (140.4, 35.4)
- added REF**: NPTH, NPTH, F.Cu at (112.1, 44.9)
- added REF**: NPTH, NPTH, F.Cu at (158.4, 89.4)
- added REF**: NPTH, NPTH, F.Cu at (156.6, 89.4)
- added REF**: NPTH, NPTH, F.Cu at (112.9, 44.9)
- added REF**: NPTH, NPTH, F.Cu at (184.1, 80.9)
- added REF**: NPTH, NPTH, F.Cu at (166.9, 97.1)
- added REF**: NPTH, NPTH, F.Cu at (112.1, 98.9)
- added REF**: NPTH, NPTH, F.Cu at (148.9, 43.1)
- added REF**: NPTH, NPTH, F.Cu at (130.9, 80.9)
- added REF**: NPTH, NPTH, F.Cu at (120.6, 89.4)
- added REF**: NPTH, NPTH, F.Cu at (158.4, 35.4)
- added REF**: NPTH, NPTH, F.Cu at (120.6, 88.6)
- added REF**: NPTH, NPTH, F.Cu at (112.9, 80.9)
- added REF**: NPTH, NPTH, F.Cu at (148.1, 79.1)
- added REF**: NPTH, NPTH, F.Cu at (192.6, 106.6)
- added REF**: NPTH, NPTH, F.Cu at (112.1, 79.1)
- added REF**: NPTH, NPTH, F.Cu at (192.6, 70.6)
- added REF**: NPTH, NPTH, F.Cu at (176.4, 89.4)
- added REF**: NPTH, NPTH, F.Cu at (158.4, 71.4)
- added REF**: NPTH, NPTH, F.Cu at (192.6, 52.6)
- added REF**: NPTH, NPTH, F.Cu at (156.6, 52.6)
- added REF**: NPTH, NPTH, F.Cu at (174.6, 89.4)
- added REF**: NPTH, NPTH, F.Cu at (166.1, 115.1)
- added REF**: NPTH, NPTH, F.Cu at (130.9, 44.9)
- added REF**: NPTH, NPTH, F.Cu at (122.4, 89.4)
- added REF**: NPTH, NPTH, F.Cu at (166.1, 98.9)
- added REF**: NPTH, NPTH, F.Cu at (148.9, 80.9)
- added REF**: Fiducial, Fiducial, F.Cu at (100.0, 22.5)
- added REF**: NPTH, NPTH, F.Cu at (140.4, 106.6)
- added REF**: NPTH, NPTH, F.Cu at (166.9, 26.9)
- added REF**: NPTH, NPTH, F.Cu at (138.6, 106.6)
- added REF**: NPTH, NPTH, F.Cu at (148.9, 98.9)
- added REF**: NPTH, NPTH, F.Cu at (112.9, 79.1)
- added REF**: NPTH, NPTH, F.Cu at (166.9, 115.1)
- added REF**: NPTH, NPTH, F.Cu at (104.4, 71.4)
- added REF**: NPTH, NPTH, F.Cu at (104.4, 70.6)
- added REF**: NPTH, NPTH, F.Cu at (174.6, 34.6)
- added REF**: NPTH, NPTH, F.Cu at (140.4, 88.6)
- added REF**: NPTH, NPTH, F.Cu at (192.6, 34.6)
- added REF**: NPTH, NPTH, F.Cu at (156.6, 34.6)
- added REF**: NPTH, NPTH, F.Cu at (166.9, 44.9)
- added REF**: NPTH, NPTH, F.Cu at (176.4, 53.4)
- added REF**: NPTH, NPTH, F.Cu at (112.9, 98.9)
- added REF**: NPTH, NPTH, F.Cu at (138.6, 71.4)
- added REF**: NPTH, NPTH, F.Cu at (112.1, 26.9)
- added REF**: NPTH, NPTH, F.Cu at (184.1, 62.9)
- added REF**: NPTH, NPTH, F.Cu at (104.4, 35.4)
- added REF**: NPTH, NPTH, F.Cu at (130.1, 44.9)
- added REF**: NPTH, NPTH, F.Cu at (184.1, 97.1)
- added REF**: NPTH, NPTH, F.Cu at (104.4, 106.6)
- added REF**: NPTH, NPTH, F.Cu at (192.6, 53.4)
- added REF**: NPTH, NPTH, F.Cu at (176.4, 52.6)
- added REF**: NPTH, NPTH, F.Cu at (138.6, 34.6)
- added REF**: NPTH, NPTH, F.Cu at (138.6, 35.4)
- added REF**: NPTH, NPTH, F.Cu at (112.1, 115.1)
- added REF**: NPTH, NPTH, F.Cu at (122.4, 70.6)
- added REF**: NPTH, NPTH, F.Cu at (174.6, 107.4)
- added REF**: NPTH, NPTH, F.Cu at (120.6, 70.6)
- added REF**: NPTH, NPTH, F.Cu at (166.9, 62.9)
- added REF**: NPTH, NPTH, F.Cu at (166.1, 26.9)
- added REF**: NPTH, NPTH, F.Cu at (184.9, 79.1)
- added REF**: NPTH, NPTH, F.Cu at (158.4, 70.6)
- added REF**: NPTH, NPTH, F.Cu at (158.4, 106.6)
- added REF**: NPTH, NPTH, F.Cu at (184.9, 61.1)
- added REF**: NPTH, NPTH, F.Cu at (184.9, 115.1)
- added REF**: NPTH, NPTH, F.Cu at (148.9, 44.9)
- added REF**: NPTH, NPTH, F.Cu at (184.1, 26.9)
- added REF**: NPTH, NPTH, F.Cu at (176.4, 71.4)
- added REF**: NPTH, NPTH, F.Cu at (130.9, 115.1)
- added REF**: NPTH, NPTH, F.Cu at (112.9, 97.1)
- added REF**: NPTH, NPTH, F.Cu at (140.4, 52.6)
- added REF**: NPTH, NPTH, F.Cu at (148.1, 80.9)
- added REF**: NPTH, NPTH, F.Cu at (174.6, 53.4)
- added REF**: NPTH, NPTH, F.Cu at (104.4, 107.4)
- added REF**: NPTH, NPTH, F.Cu at (130.1, 61.1)
- added REF**: NPTH, NPTH, F.Cu at (138.6, 53.4)
- added REF**: NPTH, NPTH, F.Cu at (156.6, 53.4)
- added REF**: Fiducial, Fiducial, B.Cu at (197.0, 22.5)
- added REF**: Fiducial, Fiducial, B.Cu at (100.0, 22.5)
- added REF**: Fiducial, Fiducial, B.Cu at (100.0, 119.5)
- added REF**: NPTH, NPTH, F.Cu at (192.6, 71.4)
- added REF**: NPTH, NPTH, F.Cu at (156.6, 70.6)
- added REF**: NPTH, NPTH, F.Cu at (184.9, 80.9)
- added REF**: NPTH, NPTH, F.Cu at (166.1, 62.9)
- added REF**: NPTH, NPTH, F.Cu at (176.4, 70.6)
- added REF**: NPTH, NPTH, F.Cu at (184.1, 61.1)
- added REF**: NPTH, NPTH, F.Cu at (148.1, 97.1)
- added REF**: NPTH, NPTH, F.Cu at (184.1, 44.9)
- added REF**: NPTH, NPTH, F.Cu at (122.4, 34.6)
- added REF**: NPTH, NPTH, F.Cu at (166.9, 61.1)
- added REF**: NPTH, NPTH, F.Cu at (158.4, 107.4)
- added REF**: NPTH, NPTH, F.Cu at (156.6, 106.6)
- added REF**: NPTH, NPTH, F.Cu at (158.4, 88.6)
- added REF**: NPTH, NPTH, F.Cu at (138.6, 88.6)
- added REF**: NPTH, NPTH, F.Cu at (112.1, 80.9)
- added REF**: NPTH, NPTH, F.Cu at (130.1, 62.9)
- added REF**: NPTH, NPTH, F.Cu at (176.4, 34.6)
- added REF**: NPTH, NPTH, F.Cu at (176.4, 35.4)
- added REF**: NPTH, NPTH, F.Cu at (140.4, 107.4)
- added REF**: NPTH, NPTH, F.Cu at (138.6, 107.4)
- added REF**: NPTH, NPTH, F.Cu at (140.4, 34.6)
- added REF**: NPTH, NPTH, F.Cu at (138.6, 89.4)
- added REF**: NPTH, NPTH, F.Cu at (166.1, 43.1)
- added REF**: NPTH, NPTH, F.Cu at (130.1, 115.1)
- added REF**: NPTH, NPTH, F.Cu at (120.6, 53.4)
- added REF**: NPTH, NPTH, F.Cu at (192.6, 88.6)
- added REF**: Fiducial, Fiducial, F.Cu at (197.0, 22.5)
- added REF**: NPTH, NPTH, F.Cu at (112.9, 115.1)
- added REF**: NPTH, NPTH, F.Cu at (130.1, 98.9)
- added REF**: NPTH, NPTH, F.Cu at (130.1, 43.1)
- added REF**: NPTH, NPTH, F.Cu at (120.6, 34.6)
- added REF**: NPTH, NPTH, F.Cu at (140.4, 53.4)
- added REF**: NPTH, NPTH, F.Cu at (148.1, 98.9)
- added REF**: NPTH, NPTH, F.Cu at (166.9, 43.1)
- added REF**: NPTH, NPTH, F.Cu at (122.4, 107.4)
- added REF**: NPTH, NPTH, F.Cu at (148.9, 62.9)
- added REF**: NPTH, NPTH, F.Cu at (140.4, 70.6)
- added REF**: NPTH, NPTH, F.Cu at (122.4, 106.6)
- added REF**: NPTH, NPTH, F.Cu at (156.6, 88.6)
- added REF**: NPTH, NPTH, F.Cu at (112.9, 26.9)
- added REF**: NPTH, NPTH, F.Cu at (130.9, 26.9)
- added REF**: NPTH, NPTH, F.Cu at (166.1, 44.9)
- added REF**: NPTH, NPTH, F.Cu at (122.4, 52.6)
- added REF**: NPTH, NPTH, F.Cu at (138.6, 52.6)
- added REF**: NPTH, NPTH, F.Cu at (138.6, 70.6)
- added REF**: NPTH, NPTH, F.Cu at (120.6, 106.6)
- added REF**: NPTH, NPTH, F.Cu at (148.9, 115.1)
- added REF**: NPTH, NPTH, F.Cu at (192.6, 35.4)
- added REF**: NPTH, NPTH, F.Cu at (130.9, 79.1)
- added REF**: NPTH, NPTH, F.Cu at (158.4, 52.6)
- added REF**: NPTH, NPTH, F.Cu at (104.4, 89.4)
- added REF**: NPTH, NPTH, F.Cu at (130.1, 80.9)
- added REF**: NPTH, NPTH, F.Cu at (112.9, 43.1)
- added REF**: NPTH, NPTH, F.Cu at (184.9, 43.1)
- added REF**: NPTH, NPTH, F.Cu at (184.9, 62.9)
- added REF**: NPTH, NPTH, F.Cu at (120.6, 35.4)
- added REF**: NPTH, NPTH, F.Cu at (184.1, 79.1)
- added REF**: NPTH, NPTH, F.Cu at (174.6, 35.4)
- added REF**: NPTH, NPTH, F.Cu at (112.1, 43.1)
- added REF**: NPTH, NPTH, F.Cu at (148.1, 61.1)
- added REF**: NPTH, NPTH, F.Cu at (176.4, 106.6)
- added REF**: NPTH, NPTH, F.Cu at (148.1, 44.9)
Other:
- outline, holes or cut-outs redrawn
