File: hardware/bno085-i2c-board-v4-panel/bno085-i2c-board-v4-panel.kicad_pcb (KiCad board)
At the start: 2 copper layers, 72 x 72 mm, 537 parts, among them J1 Conn_01x01_Pin, J2 Conn_01x01_Pin, J3 Conn_01x01_Pin, J4 Conn_01x01_Pin

Commit message: gerbers
Parts:
- removed the REF** at (115.0, 22.5) (x2)
- removed the REF** at (182.0, 22.5) (x2)
- removed the REF** at (115.0, 89.5) (x2)
- added REF**: Fiducial, Fiducial, F.Cu at (115.0, 89.5)
- added REF**: Fiducial, Fiducial, B.Cu at (115.0, 22.5)
- added REF**: Fiducial, Fiducial, B.Cu at (115.0, 89.5)
- added REF**: Fiducial, Fiducial, B.Cu at (182.0, 22.5)
- added REF**: Fiducial, Fiducial, F.Cu at (182.0, 22.5)
- added REF**: Fiducial, Fiducial, F.Cu at (115.0, 22.5)
