File: hardware/bno08x-i2c-board-v6-large/bno08x-i2c-board-v6-large.kicad_sch (KiCad schematic)
At the start: 13 parts, among them J1 PIN_SDA, J2 PIN_SCL, J3 PIN_3V3, J4 PIN_GND

Commit message: v6
Parts:
- added C3, C5: 22pF, Capacitor_SMD:C_0402_1005Metric, symbol Device:C_Small
- added Y1: 32.768kHz, Crystal:Crystal_SMD_MicroCrystal_CM9V-T1A-2Pin_1.6x1.0mm, symbol Device:Crystal_Small
Connections:
- net +3.3V: no longer U1.10 (CLKSEL0)
- net GND: now also U1.10 (CLKSEL0), C3.2, C5.2; no longer U1.26 (XOUT32/CLKSEL1)
- net XIN32: now reaches U1.27 (XIN32)
- net XIN32: now also C3.1, Y1.1
- new net CLKSEL1: C5.1, U1.26 (XOUT32/CLKSEL1), Y1.2
- no-connect marks 4 -> 3
Other:
- title: BNO08x Interface Board -> (none)
