File: hardware/bno08x-i2c-board-v6-large-crystal/bno08x-i2c-board-v6-large-crystal.kicad_pcb (KiCad board)
At the start: 2 copper layers, 16 x 16 mm, 13 parts, among them J1 PIN_SCL, J2 PIN_SDA, J3 PIN_3V3, J4 PIN_GND

Commit message: v6
Parts:
- added C4: 100nF, Capacitor_SMD:C_0402_1005Metric, F.Cu at (152.8, 78.2)
- added C5: 22pF, Capacitor_SMD:C_0402_1005Metric, F.Cu at (157.2, 80.4)
- added Y1: 32.768kHz, Crystal:Crystal_SMD_MicroCrystal_CM9V-T1A-2Pin_1.6x1.0mm, F.Cu at (155.0, 80.8)
- C3: value 100nF -> 22pF
- moved C3 2.20 mm to (152.8, 80.4), turned to 180 degrees
Connections:
- C1 pad 1: CLKSEL1 -> CLKSEL0
- C2 pad 1: CLKSEL0 -> +3.3V
- C2 pad 2: CLKSEL1 -> CLKSEL0
- C3 pad 1: CLKSEL0 -> XIN32
- C3 pad 2: CLKSEL1 -> CLKSEL0
- J3 pad 1: CLKSEL0 -> +3.3V
- J4 pad 1: CLKSEL1 -> CLKSEL0
- R1 pad 1: CLKSEL0 -> +3.3V
- R2 pad 2: CLKSEL0 -> +3.3V
- R3 pad 2: CLKSEL0 -> +3.3V
- R4 pad 2: CLKSEL0 -> +3.3V
- R5 pad 1: CLKSEL0 -> +3.3V
- U1 pad 17: CLKSEL1 -> CLKSEL0
- U1 pad 2: CLKSEL1 -> CLKSEL0
- U1 pad 25: CLKSEL1 -> CLKSEL0
- U1 pad 28: CLKSEL0 -> +3.3V
- U1 pad 3: CLKSEL0 -> +3.3V
- U1 pad 5: CLKSEL1 -> CLKSEL0
- U1 pad 6: CLKSEL1 -> CLKSEL0
Routing:
- net +3.3V: track 0.00 -> 61.0 mm, vias 0 -> 5
- net CLKSEL1: track 37.1 -> 4.15 mm, vias 2 -> 0
- net SDA: track 7.05 -> 13.6 mm, vias 0 -> 1
- net XIN32: track 0.00 -> 3.86 mm
- net Net-(U1-ENV_SCL): track 6.49 -> 5.16 mm, vias 2 -> 0
- net CLKSEL0: track 53.1 -> 52.8 mm, vias 2 -> 3
