File: hardware/bno08x-i2c-board-v6-large-crystal-panel/bno08x-i2c-board-v6-large-crystal-panel.kicad_pcb (KiCad board)
At the start: 2 copper layers, 102 x 102 mm, 794 parts, among them J1 PIN_SCL, J2 PIN_SDA, J3 PIN_3V3, J4 PIN_GND, Y1 32.768kHz

Commit message: v6 crystal
Parts:
- removed the REF** at (104.4, 89.5)
- removed the REF** at (176.4, 53.0)
- removed the REF** at (112.0, 44.9)
- removed the REF** at (158.4, 107.5)
- removed the REF** at (156.6, 53.5)
- removed the REF** at (104.5, 119.5)
- removed the REF** at (174.6, 71.5)
- removed the REF** at (99.5, 27.0)
- removed the REF** at (130.0, 98.9)
- removed the REF** at (195.0, 115.0)
- removed the REF** at (185.0, 62.9)
- removed the REF** at (197.0, 22.5) (x2)
- removed the REF** at (148.0, 80.9)
- removed the REF** at (104.5, 119.0)
- removed the REF** at (184.5, 43.1)
- removed the REF** at (158.4, 106.5)
- removed the REF** at (112.0, 79.1)
- removed the REF** at (149.0, 44.9)
- removed the REF** at (104.4, 107.5)
- removed the REF** at (122.4, 71.0)
- removed the REF** at (167.0, 97.1)
- removed the REF** at (122.4, 53.0)
- removed the REF** at (167.0, 115.1)
- removed the REF** at (122.4, 34.5)
- removed the REF** at (138.6, 89.5)
- removed the REF** at (101.5, 27.0)
- removed the REF** at (149.0, 80.9)
- removed the REF** at (167.0, 98.9)
- removed the REF** at (130.5, 115.1)
- removed the REF** at (149.0, 79.1)
- removed the REF** at (166.0, 98.9)
- removed the REF** at (130.5, 97.1)
- removed the REF** at (166.0, 61.1)
- removed the REF** at (98.0, 27.0)
- removed the REF** at (156.6, 106.5)
- removed the REF** at (104.5, 23.0)
- removed the REF** at (192.6, 107.0)
- removed the REF** at (185.0, 98.9)
- removed the REF** at (156.6, 71.0)
- removed the REF** at (156.6, 107.0)
- removed the REF** at (122.4, 52.5)
- removed the REF** at (148.5, 62.9)
- removed the REF** at (148.5, 26.9)
- removed the REF** at (166.5, 80.9)
- removed the REF** at (122.4, 70.5)
- removed the REF** at (104.5, 118.0)
- removed the REF** at (156.6, 52.5)
- removed the REF** at (120.6, 107.5)
- removed the REF** at (176.4, 89.5)
- removed the REF** at (185.0, 61.1)
- removed the REF** at (140.4, 107.5)
- removed the REF** at (130.0, 79.1)
- removed the REF** at (122.4, 107.0)
- removed the REF** at (196.0, 27.0)
- removed the REF** at (192.5, 20.5)
- removed the REF** at (104.5, 118.5)
- removed the REF** at (101.0, 27.0)
- removed the REF** at (131.0, 115.1)
- removed the REF** at (167.0, 61.1)
- removed the REF** at (192.5, 24.5)
- removed the REF** at (122.4, 35.5)
- removed the REF** at (185.0, 26.9)
- removed the REF** at (192.6, 71.0)
- removed the REF** at (174.6, 34.5)
- removed the REF** at (131.0, 26.9)
- removed the REF** at (156.6, 89.5)
- removed the REF** at (138.6, 107.5)
- removed the REF** at (138.6, 89.0)
- removed the REF** at (166.0, 44.9)
- removed the REF** at (192.6, 34.5)
- removed the REF** at (176.4, 71.5)
- removed the REF** at (174.6, 35.0)
- removed the REF** at (104.5, 120.0)
- removed the REF** at (122.4, 35.0)
- removed the REF** at (120.6, 34.5)
- removed the REF** at (195.5, 115.0)
- removed the REF** at (192.5, 120.5)
- removed the REF** at (140.4, 71.5)
- removed the REF** at (166.0, 62.9)
- removed the REF** at (112.5, 26.9)
- removed the REF** at (130.5, 62.9)
- removed the REF** at (130.5, 98.9)
- removed the REF** at (196.5, 27.0)
- removed the REF** at (112.5, 115.1)
- removed the REF** at (184.5, 62.9)
- removed the REF** at (174.6, 53.5)
- removed the REF** at (104.5, 117.5)
- removed the REF** at (176.4, 71.0)
- removed the REF** at (131.0, 43.1)
- removed the REF** at (166.5, 79.1)
- removed the REF** at (100.5, 27.0)
- removed the REF** at (192.5, 21.0)
- removed the REF** at (184.0, 62.9)
- removed the REF** at (149.0, 98.9)
- removed the REF** at (99.0, 27.0)
- removed the REF** at (176.4, 106.5)
- removed the REF** at (122.4, 89.5)
- removed the REF** at (192.5, 119.0)
- removed the REF** at (120.6, 70.5)
- removed the REF** at (113.0, 80.9)
- removed the REF** at (104.5, 21.0)
- removed the REF** at (158.4, 107.0)
- removed the REF** at (138.6, 107.0)
- removed the REF** at (112.5, 44.9)
- removed the REF** at (101.0, 115.0)
- removed the REF** at (113.0, 44.9)
- removed the REF** at (130.5, 44.9)
- removed the REF** at (130.0, 61.1)
- removed the REF** at (166.0, 26.9)
- removed the REF** at (138.6, 71.5)
- removed the REF** at (184.5, 97.1)
- removed the REF** at (166.5, 62.9)
- removed the REF** at (156.6, 34.5)
- removed the REF** at (113.0, 61.1)
- removed the REF** at (112.0, 80.9)
- removed the REF** at (120.6, 88.5)
- removed the REF** at (138.6, 52.5)
- removed the REF** at (166.0, 79.1)
- removed the REF** at (158.4, 70.5)
- removed the REF** at (192.5, 119.5)
- removed the REF** at (176.4, 53.5)
- removed the REF** at (138.6, 53.0)
- removed the REF** at (166.5, 44.9)
- removed the REF** at (140.4, 89.0)
- removed the REF** at (176.4, 35.0)
- removed the REF** at (112.0, 61.1)
- removed the REF** at (184.0, 61.1)
- removed the REF** at (149.0, 61.1)
- removed the REF** at (192.6, 53.5)
- removed the REF** at (113.0, 26.9)
- removed the REF** at (198.0, 27.0)
- removed the REF** at (148.0, 62.9)
- removed the REF** at (192.6, 71.5)
- removed the REF** at (158.4, 71.5)
- removed the REF** at (113.0, 62.9)
- removed the REF** at (199.0, 115.0)
- removed the REF** at (184.0, 44.9)
- removed the REF** at (174.6, 89.5)
- removed the REF** at (120.6, 106.5)
- removed the REF** at (166.0, 115.1)
- removed the REF** at (184.0, 80.9)
- removed the REF** at (192.6, 89.0)
- removed the REF** at (192.5, 118.5)
- removed the REF** at (148.5, 97.1)
- removed the REF** at (120.6, 53.0)
- removed the REF** at (158.4, 52.5)
- removed the REF** at (148.0, 61.1)
- removed the REF** at (104.5, 22.0)
- removed the REF** at (148.0, 26.9)
- removed the REF** at (148.0, 79.1)
- removed the REF** at (104.5, 121.5)
- removed the REF** at (184.5, 61.1)
- removed the REF** at (120.6, 89.0)
- removed the REF** at (184.0, 97.1)
- removed the REF** at (100.0, 22.5) (x2)
- removed the REF** at (131.0, 97.1)
- removed the REF** at (104.5, 21.5)
- removed the REF** at (176.4, 35.5)
- removed the REF** at (148.5, 44.9)
- removed the REF** at (104.4, 107.0)
- removed the REF** at (167.0, 43.1)
- removed the REF** at (166.0, 80.9)
- removed the REF** at (156.6, 35.0)
- removed the REF** at (158.4, 34.5)
- removed the REF** at (131.0, 79.1)
- removed the REF** at (104.4, 71.0)
- removed the REF** at (131.0, 62.9)
- removed the REF** at (140.4, 88.5)
- removed the REF** at (166.5, 61.1)
- removed the REF** at (130.0, 43.1)
- removed the REF** at (166.5, 97.1)
- removed the REF** at (148.5, 98.9)
- removed the REF** at (176.4, 88.5)
- removed the REF** at (104.5, 121.0)
- removed the REF** at (104.4, 70.5)
- removed the REF** at (174.6, 107.5)
- removed the REF** at (131.0, 98.9)
- removed the REF** at (158.4, 53.5)
- removed the REF** at (158.4, 35.0)
- removed the REF** at (122.4, 107.5)
- removed the REF** at (184.5, 26.9)
- removed the REF** at (197.5, 115.0)
- removed the REF** at (100.0, 119.5) (x2)
- removed the REF** at (140.4, 106.5)
- removed the REF** at (176.4, 52.5)
- removed the REF** at (120.6, 52.5)
- removed the REF** at (122.4, 88.5)
- removed the REF** at (112.0, 26.9)
- removed the REF** at (120.6, 89.5)
- removed the REF** at (120.6, 71.5)
- removed the REF** at (184.0, 115.1)
- removed the REF** at (192.6, 35.5)
- removed the REF** at (104.4, 89.0)
- removed the REF** at (104.4, 53.0)
- removed the REF** at (112.5, 43.1)
- removed the REF** at (174.6, 52.5)
- removed the REF** at (158.4, 88.5)
- removed the REF** at (120.6, 71.0)
- removed the REF** at (195.5, 27.0)
- removed the REF** at (184.0, 98.9)
- removed the REF** at (149.0, 43.1)
- removed the REF** at (140.4, 52.5)
- removed the REF** at (198.5, 27.0)
- removed the REF** at (100.5, 115.0)
- removed the REF** at (140.4, 34.5)
- removed the REF** at (138.6, 35.0)
- removed the REF** at (104.4, 52.5)
- removed the REF** at (112.0, 98.9)
- removed the REF** at (174.6, 88.5)
- removed the REF** at (176.4, 89.0)
- removed the REF** at (130.5, 26.9)
- removed the REF** at (138.6, 34.5)
- removed the REF** at (112.0, 97.1)
- removed the REF** at (113.0, 79.1)
- removed the REF** at (148.5, 79.1)
- removed the REF** at (100.0, 115.0)
- removed the REF** at (198.5, 115.0)
- removed the REF** at (174.6, 71.0)
- removed the REF** at (192.6, 107.5)
- removed the REF** at (104.4, 53.5)
- removed the REF** at (192.6, 52.5)
- removed the REF** at (148.5, 43.1)
- removed the REF** at (140.4, 53.5)
- removed the REF** at (104.4, 35.5)
- removed the REF** at (148.0, 44.9)
- removed the REF** at (120.6, 53.5)
- removed the REF** at (140.4, 35.5)
- removed the REF** at (130.0, 44.9)
- removed the REF** at (130.5, 43.1)
- removed the REF** at (192.5, 22.0)
- removed the REF** at (156.6, 89.0)
- removed the REF** at (195.0, 27.0)
- removed the REF** at (192.5, 118.0)
- removed the REF** at (130.0, 62.9)
- removed the REF** at (122.4, 71.5)
- removed the REF** at (99.5, 115.0)
- removed the REF** at (148.0, 98.9)
- removed the REF** at (149.0, 26.9)
- removed the REF** at (199.0, 27.0)
- removed the REF** at (130.5, 61.1)
- removed the REF** at (192.5, 117.5)
- removed the REF** at (131.0, 44.9)
- removed the REF** at (138.6, 106.5)
- removed the REF** at (140.4, 35.0)
- removed the REF** at (185.0, 80.9)
- removed the REF** at (167.0, 80.9)
- removed the REF** at (197.5, 27.0)
- removed the REF** at (174.6, 107.0)
- removed the REF** at (120.6, 35.5)
- removed the REF** at (122.4, 106.5)
- removed the REF** at (148.5, 61.1)
- removed the REF** at (104.4, 34.5)
- removed the REF** at (138.6, 53.5)
- removed the REF** at (140.4, 107.0)
- removed the REF** at (184.5, 44.9)
- removed the REF** at (166.5, 98.9)
- removed the REF** at (166.5, 26.9)
- removed the REF** at (166.5, 115.1)
- removed the REF** at (101.5, 115.0)
- removed the REF** at (112.5, 80.9)
- removed the REF** at (192.6, 70.5)
- removed the REF** at (192.5, 23.0)
- removed the REF** at (112.5, 79.1)
- removed the REF** at (98.5, 27.0)
- removed the REF** at (185.0, 44.9)
- removed the REF** at (176.4, 107.0)
- removed the REF** at (104.4, 71.5)
- removed the REF** at (138.6, 71.0)
- removed the REF** at (185.0, 97.1)
- removed the REF** at (192.5, 21.5)
- removed the REF** at (192.6, 106.5)
- removed the REF** at (176.4, 34.5)
- removed the REF** at (156.6, 107.5)
- removed the REF** at (138.6, 35.5)
- removed the REF** at (185.0, 115.1)
- removed the REF** at (130.0, 115.1)
- removed the REF** at (184.5, 80.9)
- removed the REF** at (140.4, 71.0)
- removed the REF** at (158.4, 71.0)
- removed the REF** at (192.5, 24.0)
- removed the REF** at (158.4, 89.5)
- removed the REF** at (149.0, 115.1)
- removed the REF** at (174.6, 89.0)
- removed the REF** at (104.5, 24.5)
- removed the REF** at (184.5, 98.9)
- removed the REF** at (149.0, 97.1)
- removed the REF** at (184.0, 26.9)
- removed the REF** at (156.6, 71.5)
- removed the REF** at (197.0, 115.0)
- removed the REF** at (192.5, 22.5)
- removed the REF** at (148.5, 80.9)
- removed the REF** at (148.0, 43.1)
- removed the REF** at (120.6, 107.0)
- removed the REF** at (104.4, 88.5)
- removed the REF** at (192.6, 35.0)
- removed the REF** at (99.0, 115.0)
- removed the REF** at (104.5, 22.5)
- removed the REF** at (113.0, 97.1)
- removed the REF** at (192.5, 23.5)
- removed the REF** at (174.6, 53.0)
- removed the REF** at (104.4, 35.0)
- removed the REF** at (148.0, 97.1)
- removed the REF** at (112.5, 98.9)
- removed the REF** at (184.0, 79.1)
- removed the REF** at (102.0, 27.0)
- removed the REF** at (156.6, 70.5)
- removed the REF** at (167.0, 79.1)
- removed the REF** at (184.0, 43.1)
- removed the REF** at (192.6, 53.0)
- removed the REF** at (167.0, 26.9)
- removed the REF** at (104.5, 120.5)
- removed the REF** at (156.6, 53.0)
- removed the REF** at (192.5, 121.5)
- removed the REF** at (140.4, 53.0)
- removed the REF** at (113.0, 98.9)
- removed the REF** at (140.4, 89.5)
- removed the REF** at (174.6, 35.5)
- removed the REF** at (156.6, 88.5)
- removed the REF** at (120.6, 35.0)
- removed the REF** at (130.0, 97.1)
- removed the REF** at (122.4, 53.5)
- removed the REF** at (158.4, 53.0)
- removed the REF** at (167.0, 44.9)
- removed the REF** at (184.5, 115.1)
- removed the REF** at (185.0, 43.1)
- removed the REF** at (148.0, 115.1)
- removed the REF** at (192.6, 88.5)
- removed the REF** at (104.5, 20.5)
- removed the REF** at (130.0, 80.9)
- removed the REF** at (104.5, 23.5)
- removed the REF** at (112.0, 43.1)
- removed the REF** at (112.5, 97.1)
- removed the REF** at (166.0, 97.1)
- removed the REF** at (113.0, 43.1)
- removed the REF** at (174.6, 70.5)
- removed the REF** at (192.5, 120.0)
- removed the REF** at (192.5, 121.0)
- removed the REF** at (130.5, 80.9)
- removed the REF** at (158.4, 89.0)
- removed the REF** at (196.0, 115.0)
- removed the REF** at (138.6, 70.5)
- removed the REF** at (140.4, 70.5)
- removed the REF** at (130.5, 79.1)
- removed the REF** at (185.0, 79.1)
- removed the REF** at (131.0, 61.1)
- removed the REF** at (148.5, 115.1)
- removed the REF** at (149.0, 62.9)
- removed the REF** at (166.0, 43.1)
- removed the REF** at (196.5, 115.0)
- removed the REF** at (166.5, 43.1)
- removed the REF** at (112.5, 61.1)
- removed the REF** at (112.0, 115.1)
- removed the REF** at (130.0, 26.9)
- removed the REF** at (112.0, 62.9)
- removed the REF** at (113.0, 115.1)
- removed the REF** at (184.5, 79.1)
- removed the REF** at (176.4, 107.5)
- removed the REF** at (176.4, 70.5)
- removed the REF** at (158.4, 35.5)
- removed the REF** at (167.0, 62.9)
- removed the REF** at (102.0, 115.0)
- removed the REF** at (98.5, 115.0)
- removed the REF** at (131.0, 80.9)
- removed the REF** at (104.5, 24.0)
- removed the REF** at (192.6, 89.5)
- removed the REF** at (197.0, 27.0)
- removed the REF** at (98.0, 115.0)
- removed the REF** at (174.6, 106.5)
- removed the REF** at (104.4, 106.5)
- removed the REF** at (112.5, 62.9)
- removed the REF** at (122.4, 89.0)
- removed the REF** at (100.0, 27.0)
- removed the REF** at (198.0, 115.0)
- removed the REF** at (138.6, 88.5)
- removed the REF** at (156.6, 35.5)
- added REF**: NPTH, NPTH, F.Cu at (130.2, 80.9)
- added REF**: NPTH, NPTH, F.Cu at (138.6, 107.3)
- added REF**: NPTH, NPTH, F.Cu at (112.2, 26.9)
- added REF**: NPTH, NPTH, F.Cu at (122.4, 35.3)
- added REF**: NPTH, NPTH, F.Cu at (112.2, 97.1)
- added REF**: NPTH, NPTH, F.Cu at (140.4, 88.7)
- added REF**: NPTH, NPTH, F.Cu at (112.2, 98.9)
- added REF**: NPTH, NPTH, F.Cu at (122.4, 89.3)
- added REF**: NPTH, NPTH, F.Cu at (184.2, 43.1)
- added REF**: NPTH, NPTH, F.Cu at (138.6, 70.7)
- added REF**: NPTH, NPTH, F.Cu at (99.7, 27.0)
- added REF**: NPTH, NPTH, F.Cu at (196.7, 27.0)
- added REF**: NPTH, NPTH, F.Cu at (148.2, 62.9)
- added REF**: NPTH, NPTH, F.Cu at (166.2, 62.9)
- added REF**: Fiducial, Fiducial, F.Cu at (100.0, 22.5)
- added REF**: NPTH, NPTH, F.Cu at (148.8, 97.1)
- added REF**: NPTH, NPTH, F.Cu at (130.8, 97.1)
- added REF**: NPTH, NPTH, F.Cu at (158.4, 106.7)
- added REF**: NPTH, NPTH, F.Cu at (197.8, 27.0)
- added REF**: NPTH, NPTH, F.Cu at (104.5, 22.2)
- added REF**: NPTH, NPTH, F.Cu at (184.8, 79.1)
- added REF**: NPTH, NPTH, F.Cu at (176.4, 70.7)
- added REF**: NPTH, NPTH, F.Cu at (156.6, 53.3)
- added REF**: NPTH, NPTH, F.Cu at (196.7, 115.0)
- added REF**: NPTH, NPTH, F.Cu at (174.6, 71.3)
- added REF**: NPTH, NPTH, F.Cu at (104.4, 52.7)
- added REF**: NPTH, NPTH, F.Cu at (156.6, 70.7)
- added REF**: NPTH, NPTH, F.Cu at (158.4, 89.3)
- added REF**: NPTH, NPTH, F.Cu at (156.6, 106.7)
- added REF**: NPTH, NPTH, F.Cu at (176.4, 89.3)
- added REF**: NPTH, NPTH, F.Cu at (104.5, 24.4)
- added REF**: NPTH, NPTH, F.Cu at (176.4, 106.7)
- added REF**: NPTH, NPTH, F.Cu at (184.2, 98.9)
- added REF**: NPTH, NPTH, F.Cu at (120.6, 52.7)
- added REF**: NPTH, NPTH, F.Cu at (140.4, 71.3)
- added REF**: NPTH, NPTH, F.Cu at (104.4, 89.3)
- added REF**: NPTH, NPTH, F.Cu at (104.5, 23.9)
- added REF**: NPTH, NPTH, F.Cu at (174.6, 89.3)
- added REF**: NPTH, NPTH, F.Cu at (176.4, 107.3)
- added REF**: NPTH, NPTH, F.Cu at (166.2, 61.1)
- added REF**: NPTH, NPTH, F.Cu at (192.6, 35.3)
- added REF**: NPTH, NPTH, F.Cu at (184.2, 115.1)
- added REF**: NPTH, NPTH, F.Cu at (198.9, 27.0)
- added REF**: NPTH, NPTH, F.Cu at (122.4, 53.3)
- added REF**: NPTH, NPTH, F.Cu at (140.4, 107.3)
- added REF**: NPTH, NPTH, F.Cu at (112.8, 44.9)
- added REF**: NPTH, NPTH, F.Cu at (195.6, 115.0)
- added REF**: NPTH, NPTH, F.Cu at (130.8, 43.1)
- added REF**: NPTH, NPTH, F.Cu at (156.6, 34.7)
- added REF**: NPTH, NPTH, F.Cu at (140.4, 89.3)
- added REF**: NPTH, NPTH, F.Cu at (184.8, 62.9)
- added REF**: NPTH, NPTH, F.Cu at (138.6, 53.3)
- added REF**: NPTH, NPTH, F.Cu at (192.6, 52.7)
- added REF**: NPTH, NPTH, F.Cu at (104.5, 118.7)
- added REF**: NPTH, NPTH, F.Cu at (120.6, 35.3)
- added REF**: NPTH, NPTH, F.Cu at (140.4, 35.3)
- added REF**: NPTH, NPTH, F.Cu at (130.8, 98.9)
- added REF**: NPTH, NPTH, F.Cu at (130.2, 98.9)
- added REF**: NPTH, NPTH, F.Cu at (192.6, 71.3)
- added REF**: NPTH, NPTH, F.Cu at (184.8, 26.9)
- added REF**: NPTH, NPTH, F.Cu at (192.6, 53.3)
- added REF**: NPTH, NPTH, F.Cu at (176.4, 52.7)
- added REF**: NPTH, NPTH, F.Cu at (174.6, 52.7)
- added REF**: NPTH, NPTH, F.Cu at (148.2, 44.9)
- added REF**: NPTH, NPTH, F.Cu at (166.2, 97.1)
- added REF**: NPTH, NPTH, F.Cu at (101.4, 115.0)
- added REF**: NPTH, NPTH, F.Cu at (104.4, 70.7)
- added REF**: NPTH, NPTH, F.Cu at (158.4, 35.3)
- added REF**: NPTH, NPTH, F.Cu at (166.2, 80.9)
- added REF**: NPTH, NPTH, F.Cu at (122.4, 107.3)
- added REF**: NPTH, NPTH, F.Cu at (148.2, 98.9)
- added REF**: NPTH, NPTH, F.Cu at (192.6, 107.3)
- added REF**: NPTH, NPTH, F.Cu at (120.6, 71.3)
- added REF**: NPTH, NPTH, F.Cu at (174.6, 107.3)
- added REF**: NPTH, NPTH, F.Cu at (120.6, 89.3)
- added REF**: NPTH, NPTH, F.Cu at (130.2, 44.9)
- added REF**: NPTH, NPTH, F.Cu at (122.4, 71.3)
- added REF**: NPTH, NPTH, F.Cu at (120.6, 34.7)
- added REF**: NPTH, NPTH, F.Cu at (130.2, 62.9)
- added REF**: NPTH, NPTH, F.Cu at (158.4, 34.7)
- added REF**: NPTH, NPTH, F.Cu at (138.6, 52.7)
- added REF**: NPTH, NPTH, F.Cu at (148.8, 62.9)
- added REF**: NPTH, NPTH, F.Cu at (101.4, 27.0)
- added REF**: NPTH, NPTH, F.Cu at (130.2, 43.1)
- added REF**: NPTH, NPTH, F.Cu at (130.2, 79.1)
- added REF**: NPTH, NPTH, F.Cu at (104.4, 107.3)
- added REF**: NPTH, NPTH, F.Cu at (104.4, 71.3)
- added REF**: NPTH, NPTH, F.Cu at (148.2, 80.9)
- added REF**: NPTH, NPTH, F.Cu at (99.2, 115.0)
- added REF**: NPTH, NPTH, F.Cu at (192.5, 23.3)
- added REF**: NPTH, NPTH, F.Cu at (98.1, 27.0)
- added REF**: NPTH, NPTH, F.Cu at (112.8, 62.9)
- added REF**: NPTH, NPTH, F.Cu at (148.8, 79.1)
- added REF**: NPTH, NPTH, F.Cu at (100.8, 115.0)
- added REF**: NPTH, NPTH, F.Cu at (112.8, 43.1)
- added REF**: NPTH, NPTH, F.Cu at (138.6, 106.7)
- added REF**: NPTH, NPTH, F.Cu at (197.3, 115.0)
- added REF**: NPTH, NPTH, F.Cu at (174.6, 70.7)
- added REF**: NPTH, NPTH, F.Cu at (112.2, 115.1)
- added REF**: NPTH, NPTH, F.Cu at (192.6, 34.7)
- added REF**: NPTH, NPTH, F.Cu at (184.2, 26.9)
- added REF**: NPTH, NPTH, F.Cu at (122.4, 52.7)
- added REF**: NPTH, NPTH, F.Cu at (112.2, 44.9)
- added REF**: NPTH, NPTH, F.Cu at (120.6, 107.3)
- added REF**: NPTH, NPTH, F.Cu at (148.2, 79.1)
- added REF**: NPTH, NPTH, F.Cu at (176.4, 53.3)
- added REF**: NPTH, NPTH, F.Cu at (198.4, 115.0)
- added REF**: NPTH, NPTH, F.Cu at (130.8, 79.1)
- added REF**: NPTH, NPTH, F.Cu at (197.3, 27.0)
- added REF**: NPTH, NPTH, F.Cu at (148.2, 26.9)
- added REF**: NPTH, NPTH, F.Cu at (174.6, 53.3)
- added REF**: NPTH, NPTH, F.Cu at (120.6, 70.7)
- added REF**: NPTH, NPTH, F.Cu at (184.2, 80.9)
- added REF**: NPTH, NPTH, F.Cu at (192.5, 121.4)
- added REF**: NPTH, NPTH, F.Cu at (104.4, 35.3)
- added REF**: NPTH, NPTH, F.Cu at (138.6, 35.3)
- added REF**: NPTH, NPTH, F.Cu at (156.6, 88.7)
- added REF**: NPTH, NPTH, F.Cu at (104.5, 21.7)
- added REF**: NPTH, NPTH, F.Cu at (99.7, 115.0)
- added REF**: NPTH, NPTH, F.Cu at (192.5, 119.2)
- added REF**: NPTH, NPTH, F.Cu at (184.2, 62.9)
- added REF**: NPTH, NPTH, F.Cu at (104.5, 121.4)
- added REF**: NPTH, NPTH, F.Cu at (100.8, 27.0)
- added REF**: NPTH, NPTH, F.Cu at (192.5, 117.6)
- added REF**: NPTH, NPTH, F.Cu at (130.2, 97.1)
- added REF**: NPTH, NPTH, F.Cu at (192.5, 20.6)
- added REF**: NPTH, NPTH, F.Cu at (148.8, 61.1)
- added REF**: NPTH, NPTH, F.Cu at (138.6, 89.3)
- added REF**: NPTH, NPTH, F.Cu at (166.8, 43.1)
- added REF**: NPTH, NPTH, F.Cu at (156.6, 71.3)
- added REF**: NPTH, NPTH, F.Cu at (122.4, 106.7)
- added REF**: NPTH, NPTH, F.Cu at (122.4, 70.7)
- added REF**: NPTH, NPTH, F.Cu at (130.8, 62.9)
- added REF**: NPTH, NPTH, F.Cu at (148.8, 43.1)
- added REF**: NPTH, NPTH, F.Cu at (138.6, 34.7)
- added REF**: NPTH, NPTH, F.Cu at (192.5, 22.8)
- added REF**: NPTH, NPTH, F.Cu at (195.1, 115.0)
- added REF**: NPTH, NPTH, F.Cu at (166.2, 79.1)
- added REF**: NPTH, NPTH, F.Cu at (166.2, 98.9)
- added REF**: NPTH, NPTH, F.Cu at (184.2, 79.1)
- added REF**: NPTH, NPTH, F.Cu at (104.4, 34.7)
- added REF**: NPTH, NPTH, F.Cu at (112.8, 26.9)
- added REF**: NPTH, NPTH, F.Cu at (176.4, 35.3)
- added REF**: NPTH, NPTH, F.Cu at (104.5, 118.1)
- added REF**: NPTH, NPTH, F.Cu at (112.8, 97.1)
- added REF**: NPTH, NPTH, F.Cu at (184.8, 115.1)
- added REF**: NPTH, NPTH, F.Cu at (196.2, 27.0)
- added REF**: NPTH, NPTH, F.Cu at (166.8, 62.9)
- added REF**: NPTH, NPTH, F.Cu at (130.2, 26.9)
- added REF**: NPTH, NPTH, F.Cu at (130.8, 115.1)
- added REF**: NPTH, NPTH, F.Cu at (192.5, 24.4)
- added REF**: NPTH, NPTH, F.Cu at (148.2, 43.1)
- added REF**: NPTH, NPTH, F.Cu at (112.2, 80.9)
- added REF**: NPTH, NPTH, F.Cu at (98.6, 27.0)
- added REF**: NPTH, NPTH, F.Cu at (104.5, 21.1)
- added REF**: NPTH, NPTH, F.Cu at (104.5, 20.6)
- added REF**: NPTH, NPTH, F.Cu at (104.5, 22.8)
- added REF**: NPTH, NPTH, F.Cu at (104.4, 53.3)
- added REF**: NPTH, NPTH, F.Cu at (192.5, 118.7)
- added REF**: NPTH, NPTH, F.Cu at (192.5, 120.3)
- added REF**: NPTH, NPTH, F.Cu at (192.5, 23.9)
- added REF**: NPTH, NPTH, F.Cu at (130.8, 80.9)
- added REF**: NPTH, NPTH, F.Cu at (192.6, 89.3)
- added REF**: NPTH, NPTH, F.Cu at (120.6, 53.3)
- added REF**: NPTH, NPTH, F.Cu at (184.2, 61.1)
- added REF**: NPTH, NPTH, F.Cu at (148.8, 26.9)
- added REF**: NPTH, NPTH, F.Cu at (112.8, 61.1)
- added REF**: NPTH, NPTH, F.Cu at (130.2, 115.1)
- added REF**: NPTH, NPTH, F.Cu at (112.2, 61.1)
- added REF**: NPTH, NPTH, F.Cu at (122.4, 34.7)
- added REF**: NPTH, NPTH, F.Cu at (122.4, 88.7)
- added REF**: NPTH, NPTH, F.Cu at (192.5, 119.8)
- added REF**: NPTH, NPTH, F.Cu at (120.6, 106.7)
- added REF**: NPTH, NPTH, F.Cu at (192.5, 120.9)
- added REF**: NPTH, NPTH, F.Cu at (192.6, 88.7)
- added REF**: NPTH, NPTH, F.Cu at (184.8, 43.1)
- added REF**: NPTH, NPTH, F.Cu at (148.8, 115.1)
- added REF**: NPTH, NPTH, F.Cu at (192.5, 118.1)
- added REF**: NPTH, NPTH, F.Cu at (192.5, 22.2)
- added REF**: NPTH, NPTH, F.Cu at (166.2, 115.1)
- added REF**: NPTH, NPTH, F.Cu at (156.6, 107.3)
- added REF**: NPTH, NPTH, F.Cu at (140.4, 52.7)
- added REF**: NPTH, NPTH, F.Cu at (148.2, 115.1)
- added REF**: NPTH, NPTH, F.Cu at (195.6, 27.0)
- added REF**: NPTH, NPTH, F.Cu at (130.2, 61.1)
- added REF**: NPTH, NPTH, F.Cu at (140.4, 106.7)
- added REF**: NPTH, NPTH, F.Cu at (166.2, 44.9)
- added REF**: NPTH, NPTH, F.Cu at (156.6, 52.7)
- added REF**: NPTH, NPTH, F.Cu at (166.8, 79.1)
- added REF**: NPTH, NPTH, F.Cu at (148.8, 98.9)
- added REF**: NPTH, NPTH, F.Cu at (148.2, 97.1)
- added REF**: NPTH, NPTH, F.Cu at (101.9, 27.0)
- added REF**: NPTH, NPTH, F.Cu at (112.2, 62.9)
- added REF**: NPTH, NPTH, F.Cu at (192.6, 106.7)
- added REF**: NPTH, NPTH, F.Cu at (112.8, 80.9)
- added REF**: Fiducial, Fiducial, B.Cu at (197.0, 22.5)
- added REF**: Fiducial, Fiducial, B.Cu at (100.0, 22.5)
- added REF**: Fiducial, Fiducial, B.Cu at (100.0, 119.5)
- added REF**: NPTH, NPTH, F.Cu at (197.8, 115.0)
- added REF**: NPTH, NPTH, F.Cu at (184.8, 61.1)
- added REF**: NPTH, NPTH, F.Cu at (140.4, 70.7)
- added REF**: NPTH, NPTH, F.Cu at (195.1, 27.0)
- added REF**: Fiducial, Fiducial, F.Cu at (100.0, 119.5)
- added REF**: NPTH, NPTH, F.Cu at (184.2, 44.9)
- added REF**: NPTH, NPTH, F.Cu at (184.8, 44.9)
- added REF**: NPTH, NPTH, F.Cu at (166.8, 97.1)
- added REF**: NPTH, NPTH, F.Cu at (158.4, 70.7)
- added REF**: NPTH, NPTH, F.Cu at (104.4, 106.7)
- added REF**: NPTH, NPTH, F.Cu at (166.8, 80.9)
- added REF**: NPTH, NPTH, F.Cu at (166.8, 61.1)
- added REF**: NPTH, NPTH, F.Cu at (112.2, 43.1)
- added REF**: NPTH, NPTH, F.Cu at (138.6, 71.3)
- added REF**: NPTH, NPTH, F.Cu at (198.4, 27.0)
- added REF**: NPTH, NPTH, F.Cu at (156.6, 35.3)
- added REF**: NPTH, NPTH, F.Cu at (184.2, 97.1)
- added REF**: NPTH, NPTH, F.Cu at (174.6, 34.7)
- added REF**: NPTH, NPTH, F.Cu at (140.4, 53.3)
- added REF**: NPTH, NPTH, F.Cu at (112.2, 79.1)
- added REF**: NPTH, NPTH, F.Cu at (192.5, 21.1)
- added REF**: NPTH, NPTH, F.Cu at (138.6, 88.7)
- added REF**: NPTH, NPTH, F.Cu at (104.5, 119.8)
- added REF**: NPTH, NPTH, F.Cu at (198.9, 115.0)
- added REF**: NPTH, NPTH, F.Cu at (174.6, 106.7)
- added REF**: NPTH, NPTH, F.Cu at (174.6, 35.3)
- added REF**: NPTH, NPTH, F.Cu at (130.8, 26.9)
- added REF**: NPTH, NPTH, F.Cu at (130.8, 61.1)
- added REF**: NPTH, NPTH, F.Cu at (166.8, 115.1)
- added REF**: NPTH, NPTH, F.Cu at (104.5, 23.3)
- added REF**: NPTH, NPTH, F.Cu at (104.4, 88.7)
- added REF**: NPTH, NPTH, F.Cu at (158.4, 107.3)
- added REF**: NPTH, NPTH, F.Cu at (156.6, 89.3)
- added REF**: NPTH, NPTH, F.Cu at (104.5, 119.2)
- added REF**: NPTH, NPTH, F.Cu at (192.5, 21.7)
- added REF**: NPTH, NPTH, F.Cu at (140.4, 34.7)
- added REF**: NPTH, NPTH, F.Cu at (176.4, 88.7)
- added REF**: NPTH, NPTH, F.Cu at (112.8, 79.1)
- added REF**: NPTH, NPTH, F.Cu at (184.8, 80.9)
- added REF**: NPTH, NPTH, F.Cu at (184.8, 98.9)
- added REF**: Fiducial, Fiducial, F.Cu at (197.0, 22.5)
- added REF**: NPTH, NPTH, F.Cu at (176.4, 71.3)
- added REF**: NPTH, NPTH, F.Cu at (148.2, 61.1)
- added REF**: NPTH, NPTH, F.Cu at (101.9, 115.0)
- added REF**: NPTH, NPTH, F.Cu at (112.8, 115.1)
- added REF**: NPTH, NPTH, F.Cu at (100.3, 27.0)
- added REF**: NPTH, NPTH, F.Cu at (120.6, 88.7)
- added REF**: NPTH, NPTH, F.Cu at (166.8, 26.9)
- added REF**: NPTH, NPTH, F.Cu at (158.4, 52.7)
- added REF**: NPTH, NPTH, F.Cu at (104.5, 120.3)
- added REF**: NPTH, NPTH, F.Cu at (166.8, 44.9)
- added REF**: NPTH, NPTH, F.Cu at (99.2, 27.0)
- added REF**: NPTH, NPTH, F.Cu at (112.8, 98.9)
- added REF**: NPTH, NPTH, F.Cu at (166.2, 26.9)
- added REF**: NPTH, NPTH, F.Cu at (166.2, 43.1)
- added REF**: NPTH, NPTH, F.Cu at (174.6, 88.7)
- added REF**: NPTH, NPTH, F.Cu at (100.3, 115.0)
- added REF**: NPTH, NPTH, F.Cu at (196.2, 115.0)
- added REF**: NPTH, NPTH, F.Cu at (158.4, 71.3)
- added REF**: NPTH, NPTH, F.Cu at (158.4, 53.3)
- added REF**: NPTH, NPTH, F.Cu at (176.4, 34.7)
- added REF**: NPTH, NPTH, F.Cu at (192.6, 70.7)
- added REF**: NPTH, NPTH, F.Cu at (130.8, 44.9)
- added REF**: NPTH, NPTH, F.Cu at (98.1, 115.0)
- added REF**: NPTH, NPTH, F.Cu at (184.8, 97.1)
- added REF**: NPTH, NPTH, F.Cu at (166.8, 98.9)
- added REF**: NPTH, NPTH, F.Cu at (148.8, 44.9)
- added REF**: NPTH, NPTH, F.Cu at (148.8, 80.9)
- added REF**: NPTH, NPTH, F.Cu at (158.4, 88.7)
- added REF**: NPTH, NPTH, F.Cu at (104.5, 117.6)
- added REF**: NPTH, NPTH, F.Cu at (98.6, 115.0)
- added REF**: NPTH, NPTH, F.Cu at (104.5, 120.9)
