File: hardware/bno08x-i2c-board-v6-panel/bno08x-i2c-board-v6-panel.kicad_pcb (KiCad board)
At the start: 2 copper layers, 75.5 x 75.5 mm, 719 parts, among them J1 PIN_SCL, J2 PIN_SDA, J3 PIN_3V3, J4 PIN_GND

Commit message: v6 crystal
Parts:
- removed the REF** at (179.2, 21.5)
- removed the REF** at (114.3, 88.5)
- removed the REF** at (128.6, 45.0)
- removed the REF** at (161.2, 65.0)
- removed the REF** at (136.3, 88.6)
- removed the REF** at (143.0, 32.3)
- removed the REF** at (117.7, 82.6)
- removed the REF** at (166.6, 45.6)
- removed the REF** at (174.4, 52.3)
- removed the REF** at (160.7, 26.9)
- removed the REF** at (148.0, 88.6)
- removed the REF** at (117.8, 95.0)
- removed the REF** at (155.7, 32.3)
- removed the REF** at (135.8, 77.7)
- removed the REF** at (173.4, 63.2)
- removed the REF** at (143.1, 69.9)
- removed the REF** at (135.3, 26.9)
- removed the REF** at (179.2, 91.0)
- removed the REF** at (155.8, 82.6)
- removed the REF** at (161.2, 88.6)
- removed the REF** at (185.7, 27.0)
- removed the REF** at (154.0, 57.7)
- removed the REF** at (117.7, 44.5)
- removed the REF** at (166.6, 32.9)
- removed the REF** at (123.1, 26.9)
- removed the REF** at (179.2, 22.5)
- removed the REF** at (179.2, 92.5)
- removed the REF** at (111.3, 27.0)
- removed the REF** at (123.6, 77.7)
- removed the REF** at (123.6, 63.2)
- removed the REF** at (173.9, 65.0)
- removed the REF** at (173.4, 65.0)
- removed the REF** at (122.6, 50.5)
- removed the REF** at (141.2, 45.6)
- removed the REF** at (117.7, 69.9)
- removed the REF** at (179.2, 21.0)
- removed the REF** at (168.5, 44.5)
- removed the REF** at (123.1, 52.3)
- removed the REF** at (161.7, 50.5)
- removed the REF** at (148.5, 37.8)
- removed the REF** at (173.9, 63.2)
- removed the REF** at (122.6, 88.6)
- removed the REF** at (173.4, 50.5)
- removed the REF** at (128.5, 45.6)
- removed the REF** at (135.3, 39.6)
- removed the REF** at (155.7, 70.4)
- removed the REF** at (179.2, 20.5)
- removed the REF** at (143.1, 31.8)
- removed the REF** at (155.7, 57.7)
- removed the REF** at (136.3, 63.2)
- removed the REF** at (114.3, 27.0)
- removed the REF** at (123.1, 65.0)
- removed the REF** at (135.8, 50.5)
- removed the REF** at (173.4, 26.9)
- removed the REF** at (161.7, 39.6)
- removed the REF** at (117.8, 21.0)
- removed the REF** at (141.3, 57.7)
- removed the REF** at (135.8, 52.3)
- removed the REF** at (155.8, 83.7)
- removed the REF** at (166.7, 70.4)
- removed the REF** at (114.8, 88.5)
- removed the REF** at (123.1, 37.8)
- removed the REF** at (173.9, 39.6)
- removed the REF** at (148.0, 65.0)
- removed the REF** at (123.6, 26.9)
- removed the REF** at (160.7, 39.6)
- removed the REF** at (173.9, 50.5)
- removed the REF** at (160.7, 88.6)
- removed the REF** at (153.9, 71.0)
- removed the REF** at (113.8, 27.0)
- removed the REF** at (179.2, 91.5)
- removed the REF** at (117.8, 20.5)
- removed the REF** at (148.5, 39.6)
- removed the REF** at (153.9, 57.2)
- removed the REF** at (166.6, 44.5)
- removed the REF** at (122.6, 65.0)
- removed the REF** at (174.4, 65.0)
- removed the REF** at (123.6, 52.3)
- removed the REF** at (155.8, 45.6)
- removed the REF** at (136.3, 75.9)
- removed the REF** at (153.9, 83.7)
- removed the REF** at (179.3, 83.7)
- removed the REF** at (122.6, 52.3)
- removed the REF** at (135.8, 26.9)
- removed the REF** at (117.6, 70.4)
- removed the REF** at (148.0, 77.7)
- removed the REF** at (179.2, 24.0)
- removed the REF** at (141.3, 32.3)
- removed the REF** at (135.3, 52.3)
- removed the REF** at (130.3, 57.7)
- removed the REF** at (143.1, 71.0)
- removed the REF** at (166.6, 57.2)
- removed the REF** at (112.3, 27.0)
- removed the REF** at (128.6, 70.4)
- removed the REF** at (184.7, 27.0)
- removed the REF** at (123.1, 88.6)
- removed the REF** at (128.5, 69.9)
- removed the REF** at (161.2, 77.7)
- removed the REF** at (174.4, 50.5)
- removed the REF** at (117.7, 58.3)
- removed the REF** at (111.8, 27.0)
- removed the REF** at (155.8, 58.3)
- removed the REF** at (130.4, 45.6)
- removed the REF** at (136.3, 77.7)
- removed the REF** at (179.3, 69.9)
- removed the REF** at (135.3, 88.6)
- removed the REF** at (148.5, 50.5)
- removed the REF** at (117.8, 23.5)
- removed the REF** at (166.6, 83.7)
- removed the REF** at (143.1, 83.7)
- removed the REF** at (130.4, 69.9)
- removed the REF** at (122.6, 63.2)
- removed the REF** at (154.0, 83.1)
- removed the REF** at (168.4, 32.3)
- removed the REF** at (153.9, 45.6)
- removed the REF** at (113.3, 93.0) (x2)
- removed the REF** at (141.2, 69.9)
- removed the REF** at (183.7, 27.0)
- removed the REF** at (182.7, 27.0)
- removed the REF** at (128.6, 83.1)
- removed the REF** at (179.2, 92.0)
- removed the REF** at (160.7, 65.0)
- removed the REF** at (179.4, 57.7)
- removed the REF** at (161.7, 37.8)
- removed the REF** at (111.8, 88.5)
- removed the REF** at (114.8, 27.0)
- removed the REF** at (168.5, 83.7)
- removed the REF** at (161.7, 77.7)
- removed the REF** at (135.8, 88.6)
- removed the REF** at (148.0, 37.8)
- removed the REF** at (161.2, 52.3)
- removed the REF** at (113.3, 27.0)
- removed the REF** at (179.2, 95.0)
- removed the REF** at (135.3, 63.2)
- removed the REF** at (123.6, 39.6)
- removed the REF** at (143.0, 70.4)
- removed the REF** at (161.2, 26.9)
- removed the REF** at (153.9, 82.6)
- removed the REF** at (143.1, 57.2)
- removed the REF** at (168.5, 69.9)
- removed the REF** at (160.7, 52.3)
- removed the REF** at (161.2, 63.2)
- removed the REF** at (179.4, 83.1)
- removed the REF** at (161.2, 37.8)
- removed the REF** at (123.1, 39.6)
- removed the REF** at (173.9, 88.6)
- removed the REF** at (155.8, 71.0)
- removed the REF** at (130.4, 31.8)
- removed the REF** at (182.7, 88.5)
- removed the REF** at (179.4, 32.3)
- removed the REF** at (174.4, 63.2)
- removed the REF** at (117.8, 93.5)
- removed the REF** at (166.6, 31.8)
- removed the REF** at (154.0, 32.3)
- removed the REF** at (168.4, 70.4)
- removed the REF** at (128.5, 44.5)
- removed the REF** at (141.3, 45.0)
- removed the REF** at (166.6, 82.6)
- removed the REF** at (128.5, 82.6)
- removed the REF** at (117.8, 23.0)
- removed the REF** at (168.4, 57.7)
- removed the REF** at (149.0, 52.3)
- removed the REF** at (174.4, 37.8)
- removed the REF** at (149.0, 50.5)
- removed the REF** at (179.2, 94.5)
- removed the REF** at (148.0, 50.5)
- removed the REF** at (179.2, 22.0)
- removed the REF** at (168.5, 82.6)
- removed the REF** at (117.7, 71.0)
- removed the REF** at (155.8, 44.5)
- removed the REF** at (174.4, 88.6)
- removed the REF** at (135.8, 75.9)
- removed the REF** at (135.3, 37.8)
- removed the REF** at (168.5, 58.3)
- removed the REF** at (160.7, 75.9)
- removed the REF** at (160.7, 37.8)
- removed the REF** at (184.2, 27.0)
- removed the REF** at (166.6, 69.9)
- removed the REF** at (149.0, 75.9)
- removed the REF** at (166.7, 57.7)
- removed the REF** at (136.3, 50.5)
- removed the REF** at (123.1, 50.5)
- removed the REF** at (161.2, 39.6)
- removed the REF** at (149.0, 65.0)
- removed the REF** at (122.6, 77.7)
- removed the REF** at (179.3, 71.0)
- removed the REF** at (141.3, 83.1)
- removed the REF** at (184.2, 88.5)
- removed the REF** at (117.8, 21.5)
- removed the REF** at (130.3, 45.0)
- removed the REF** at (143.1, 44.5)
- removed the REF** at (179.3, 82.6)
- removed the REF** at (183.2, 27.0)
- removed the REF** at (179.2, 94.0)
- removed the REF** at (149.0, 77.7)
- removed the REF** at (168.5, 71.0)
- removed the REF** at (111.3, 88.5)
- removed the REF** at (154.0, 45.0)
- removed the REF** at (161.2, 75.9)
- removed the REF** at (148.0, 52.3)
- removed the REF** at (181.7, 27.0)
- removed the REF** at (143.0, 83.1)
- removed the REF** at (112.3, 88.5)
- removed the REF** at (136.3, 26.9)
- removed the REF** at (148.5, 75.9)
- removed the REF** at (117.8, 91.0)
- removed the REF** at (135.8, 39.6)
- removed the REF** at (166.7, 32.3)
- removed the REF** at (168.5, 31.8)
- removed the REF** at (117.8, 22.0)
- removed the REF** at (113.3, 88.5)
- removed the REF** at (130.3, 83.1)
- removed the REF** at (136.3, 52.3)
- removed the REF** at (149.0, 88.6)
- removed the REF** at (123.6, 50.5)
- removed the REF** at (166.7, 83.1)
- removed the REF** at (135.3, 50.5)
- removed the REF** at (130.3, 32.3)
- removed the REF** at (168.4, 83.1)
- removed the REF** at (128.5, 83.7)
- removed the REF** at (166.7, 45.0)
- removed the REF** at (128.5, 58.3)
- removed the REF** at (174.4, 77.7)
- removed the REF** at (123.6, 75.9)
- removed the REF** at (160.7, 50.5)
- removed the REF** at (135.8, 37.8)
- removed the REF** at (149.0, 39.6)
- removed the REF** at (179.2, 23.5)
- removed the REF** at (179.3, 58.3)
- removed the REF** at (160.7, 77.7)
- removed the REF** at (128.5, 71.0)
- removed the REF** at (148.5, 65.0)
- removed the REF** at (117.8, 93.0)
- removed the REF** at (141.2, 71.0)
- removed the REF** at (130.4, 71.0)
- removed the REF** at (148.5, 63.2)
- removed the REF** at (117.7, 45.6)
- removed the REF** at (174.4, 26.9)
- removed the REF** at (148.0, 63.2)
- removed the REF** at (155.8, 31.8)
- removed the REF** at (168.5, 32.9)
- removed the REF** at (128.5, 57.2)
- removed the REF** at (183.2, 88.5)
- removed the REF** at (130.4, 44.5)
- removed the REF** at (141.2, 83.7)
- removed the REF** at (161.7, 75.9)
- removed the REF** at (141.2, 32.9)
- removed the REF** at (117.7, 57.2)
- removed the REF** at (155.8, 69.9)
- removed the REF** at (130.4, 57.2)
- removed the REF** at (166.6, 58.3)
- removed the REF** at (113.8, 88.5)
- removed the REF** at (122.6, 39.6)
- removed the REF** at (141.2, 57.2)
- removed the REF** at (174.4, 39.6)
- removed the REF** at (185.7, 88.5)
- removed the REF** at (123.6, 88.6)
- removed the REF** at (173.4, 39.6)
- removed the REF** at (143.1, 45.6)
- removed the REF** at (183.7, 22.5) (x2)
- removed the REF** at (130.4, 32.9)
- removed the REF** at (185.2, 27.0)
- removed the REF** at (154.0, 70.4)
- removed the REF** at (148.0, 26.9)
- removed the REF** at (143.1, 82.6)
- removed the REF** at (141.2, 31.8)
- removed the REF** at (123.6, 65.0)
- removed the REF** at (122.6, 26.9)
- removed the REF** at (112.8, 88.5)
- removed the REF** at (179.3, 31.8)
- removed the REF** at (173.9, 77.7)
- removed the REF** at (173.9, 52.3)
- removed the REF** at (143.0, 45.0)
- removed the REF** at (153.9, 44.5)
- removed the REF** at (117.8, 94.5)
- removed the REF** at (182.2, 88.5)
- removed the REF** at (135.3, 75.9)
- removed the REF** at (149.0, 26.9)
- removed the REF** at (179.4, 45.0)
- removed the REF** at (117.7, 83.7)
- removed the REF** at (179.2, 24.5)
- removed the REF** at (179.4, 70.4)
- removed the REF** at (179.3, 45.6)
- removed the REF** at (161.7, 88.6)
- removed the REF** at (183.7, 88.5)
- removed the REF** at (141.3, 70.4)
- removed the REF** at (182.2, 27.0)
- removed the REF** at (117.6, 45.0)
- removed the REF** at (128.5, 31.8)
- removed the REF** at (136.3, 39.6)
- removed the REF** at (179.3, 32.9)
- removed the REF** at (153.9, 32.9)
- removed the REF** at (148.5, 88.6)
- removed the REF** at (143.0, 57.7)
- removed the REF** at (128.5, 32.9)
- removed the REF** at (117.8, 24.0)
- removed the REF** at (141.2, 58.3)
- removed the REF** at (173.9, 37.8)
- removed the REF** at (117.7, 32.9)
- removed the REF** at (155.8, 57.2)
- removed the REF** at (117.8, 92.0)
- removed the REF** at (161.7, 26.9)
- removed the REF** at (181.7, 88.5)
- removed the REF** at (148.5, 26.9)
- removed the REF** at (123.1, 63.2)
- removed the REF** at (141.2, 82.6)
- removed the REF** at (185.2, 88.5)
- removed the REF** at (174.4, 75.9)
- removed the REF** at (122.6, 75.9)
- removed the REF** at (173.4, 52.3)
- removed the REF** at (155.7, 45.0)
- removed the REF** at (168.5, 57.2)
- removed the REF** at (173.4, 75.9)
- removed the REF** at (113.3, 22.5) (x2)
- removed the REF** at (143.1, 58.3)
- removed the REF** at (115.3, 27.0)
- removed the REF** at (149.0, 63.2)
- removed the REF** at (179.2, 93.5)
- removed the REF** at (148.5, 52.3)
- removed the REF** at (173.4, 37.8)
- removed the REF** at (179.2, 23.0)
- removed the REF** at (117.8, 22.5)
- removed the REF** at (148.0, 75.9)
- removed the REF** at (115.3, 88.5)
- removed the REF** at (130.4, 82.6)
- removed the REF** at (161.2, 50.5)
- removed the REF** at (160.7, 63.2)
- removed the REF** at (155.7, 83.1)
- removed the REF** at (122.6, 37.8)
- removed the REF** at (173.4, 88.6)
- removed the REF** at (130.3, 70.4)
- removed the REF** at (135.8, 65.0)
- removed the REF** at (117.8, 91.5)
- removed the REF** at (130.4, 83.7)
- removed the REF** at (168.4, 45.0)
- removed the REF** at (123.1, 77.7)
- removed the REF** at (128.6, 32.3)
- removed the REF** at (173.4, 77.7)
- removed the REF** at (123.6, 37.8)
- removed the REF** at (112.8, 27.0)
- removed the REF** at (161.7, 65.0)
- removed the REF** at (117.6, 32.3)
- removed the REF** at (136.3, 65.0)
- removed the REF** at (153.9, 58.3)
- removed the REF** at (117.6, 57.7)
- removed the REF** at (179.3, 57.2)
- removed the REF** at (153.9, 31.8)
- removed the REF** at (166.6, 71.0)
- removed the REF** at (161.7, 52.3)
- removed the REF** at (117.6, 83.1)
- removed the REF** at (117.8, 92.5)
- removed the REF** at (117.8, 94.0)
- removed the REF** at (148.0, 39.6)
- removed the REF** at (117.7, 31.8)
- removed the REF** at (153.9, 69.9)
- removed the REF** at (173.9, 75.9)
- removed the REF** at (149.0, 37.8)
- removed the REF** at (136.3, 37.8)
- removed the REF** at (117.8, 24.5)
- removed the REF** at (161.7, 63.2)
- removed the REF** at (130.4, 58.3)
- removed the REF** at (135.8, 63.2)
- removed the REF** at (173.9, 26.9)
- removed the REF** at (155.8, 32.9)
- removed the REF** at (143.1, 32.9)
- removed the REF** at (179.3, 44.5)
- removed the REF** at (135.3, 77.7)
- removed the REF** at (141.2, 44.5)
- removed the REF** at (168.5, 45.6)
- removed the REF** at (135.3, 65.0)
- removed the REF** at (179.2, 93.0)
- removed the REF** at (128.6, 57.7)
- removed the REF** at (184.7, 88.5)
- removed the REF** at (123.1, 75.9)
- removed the REF** at (148.5, 77.7)
- added REF**: NPTH, NPTH, F.Cu at (179.2, 92.7)
- added REF**: NPTH, NPTH, F.Cu at (154.0, 83.5)
- added REF**: NPTH, NPTH, F.Cu at (136.1, 65.0)
- added REF**: NPTH, NPTH, F.Cu at (112.4, 88.5)
- added REF**: NPTH, NPTH, F.Cu at (161.5, 26.9)
- added REF**: NPTH, NPTH, F.Cu at (179.2, 22.2)
- added REF**: NPTH, NPTH, F.Cu at (148.8, 39.6)
- added REF**: NPTH, NPTH, F.Cu at (117.6, 83.5)
- added REF**: NPTH, NPTH, F.Cu at (174.2, 63.2)
- added REF**: NPTH, NPTH, F.Cu at (123.4, 26.9)
- added REF**: NPTH, NPTH, F.Cu at (117.8, 91.1)
- added REF**: NPTH, NPTH, F.Cu at (115.2, 88.5)
- added REF**: NPTH, NPTH, F.Cu at (161.5, 65.0)
- added REF**: NPTH, NPTH, F.Cu at (113.5, 27.0)
- added REF**: NPTH, NPTH, F.Cu at (160.9, 52.3)
- added REF**: NPTH, NPTH, F.Cu at (128.6, 45.4)
- added REF**: NPTH, NPTH, F.Cu at (128.6, 57.4)
- added REF**: NPTH, NPTH, F.Cu at (123.4, 88.6)
- added REF**: NPTH, NPTH, F.Cu at (179.4, 83.5)
- added REF**: NPTH, NPTH, F.Cu at (123.4, 65.0)
- added REF**: NPTH, NPTH, F.Cu at (179.2, 94.9)
- added REF**: NPTH, NPTH, F.Cu at (135.5, 75.9)
- added REF**: NPTH, NPTH, F.Cu at (154.0, 44.7)
- added REF**: NPTH, NPTH, F.Cu at (117.8, 22.2)
- added REF**: NPTH, NPTH, F.Cu at (168.4, 83.5)
- added REF**: NPTH, NPTH, F.Cu at (148.8, 26.9)
- added REF**: NPTH, NPTH, F.Cu at (174.2, 65.0)
- added REF**: NPTH, NPTH, F.Cu at (179.2, 24.4)
- added REF**: NPTH, NPTH, F.Cu at (143.0, 32.7)
- added REF**: NPTH, NPTH, F.Cu at (111.9, 27.0)
- added REF**: NPTH, NPTH, F.Cu at (117.6, 44.7)
- added REF**: NPTH, NPTH, F.Cu at (184.6, 88.5)
- added REF**: NPTH, NPTH, F.Cu at (111.3, 88.5)
- added REF**: NPTH, NPTH, F.Cu at (117.8, 92.2)
- added REF**: NPTH, NPTH, F.Cu at (130.3, 58.1)
- added REF**: NPTH, NPTH, F.Cu at (168.4, 82.8)
- added REF**: NPTH, NPTH, F.Cu at (128.6, 32.7)
- added REF**: NPTH, NPTH, F.Cu at (111.3, 27.0)
- added REF**: NPTH, NPTH, F.Cu at (117.6, 57.4)
- added REF**: NPTH, NPTH, F.Cu at (168.4, 57.4)
- added REF**: NPTH, NPTH, F.Cu at (179.4, 44.7)
- added REF**: NPTH, NPTH, F.Cu at (179.4, 70.1)
- added REF**: NPTH, NPTH, F.Cu at (155.7, 58.1)
- added REF**: NPTH, NPTH, F.Cu at (141.3, 58.1)
- added REF**: NPTH, NPTH, F.Cu at (130.3, 70.8)
- added REF**: NPTH, NPTH, F.Cu at (168.4, 70.8)
- added REF**: NPTH, NPTH, F.Cu at (148.2, 39.6)
- added REF**: NPTH, NPTH, F.Cu at (117.8, 21.7)
- added REF**: NPTH, NPTH, F.Cu at (148.2, 88.6)
- added REF**: NPTH, NPTH, F.Cu at (160.9, 39.6)
- added REF**: NPTH, NPTH, F.Cu at (122.8, 75.9)
- added REF**: NPTH, NPTH, F.Cu at (128.6, 58.1)
- added REF**: NPTH, NPTH, F.Cu at (155.7, 83.5)
- added REF**: NPTH, NPTH, F.Cu at (148.2, 63.2)
- added REF**: NPTH, NPTH, F.Cu at (179.4, 82.8)
- added REF**: NPTH, NPTH, F.Cu at (117.8, 93.8)
- added REF**: NPTH, NPTH, F.Cu at (135.5, 52.3)
- added REF**: NPTH, NPTH, F.Cu at (182.9, 27.0)
- added REF**: NPTH, NPTH, F.Cu at (160.9, 65.0)
- added REF**: NPTH, NPTH, F.Cu at (182.9, 88.5)
- added REF**: NPTH, NPTH, F.Cu at (135.5, 88.6)
- added REF**: NPTH, NPTH, F.Cu at (160.9, 50.5)
- added REF**: NPTH, NPTH, F.Cu at (117.6, 70.1)
- added REF**: NPTH, NPTH, F.Cu at (166.7, 83.5)
- added REF**: NPTH, NPTH, F.Cu at (117.8, 21.1)
- added REF**: NPTH, NPTH, F.Cu at (128.6, 70.1)
- added REF**: NPTH, NPTH, F.Cu at (161.5, 88.6)
- added REF**: NPTH, NPTH, F.Cu at (117.8, 23.3)
- added REF**: Fiducial, Fiducial, F.Cu at (113.3, 22.5)
- added REF**: NPTH, NPTH, F.Cu at (114.1, 27.0)
- added REF**: NPTH, NPTH, F.Cu at (155.7, 32.0)
- added REF**: Fiducial, Fiducial, F.Cu at (183.7, 22.5)
- added REF**: NPTH, NPTH, F.Cu at (148.2, 37.8)
- added REF**: NPTH, NPTH, F.Cu at (182.4, 88.5)
- added REF**: NPTH, NPTH, F.Cu at (173.6, 88.6)
- added REF**: NPTH, NPTH, F.Cu at (166.7, 70.8)
- added REF**: NPTH, NPTH, F.Cu at (130.3, 83.5)
- added REF**: NPTH, NPTH, F.Cu at (128.6, 83.5)
- added REF**: NPTH, NPTH, F.Cu at (184.0, 88.5)
- added REF**: NPTH, NPTH, F.Cu at (148.2, 26.9)
- added REF**: NPTH, NPTH, F.Cu at (161.5, 37.8)
- added REF**: NPTH, NPTH, F.Cu at (141.3, 45.4)
- added REF**: NPTH, NPTH, F.Cu at (111.9, 88.5)
- added REF**: NPTH, NPTH, F.Cu at (148.2, 65.0)
- added REF**: NPTH, NPTH, F.Cu at (154.0, 32.7)
- added REF**: NPTH, NPTH, F.Cu at (117.8, 94.4)
- added REF**: NPTH, NPTH, F.Cu at (166.7, 57.4)
- added REF**: NPTH, NPTH, F.Cu at (179.2, 23.9)
- added REF**: NPTH, NPTH, F.Cu at (130.3, 82.8)
- added REF**: NPTH, NPTH, F.Cu at (136.1, 52.3)
- added REF**: NPTH, NPTH, F.Cu at (117.8, 22.8)
- added REF**: NPTH, NPTH, F.Cu at (174.2, 39.6)
- added REF**: NPTH, NPTH, F.Cu at (117.8, 93.3)
- added REF**: NPTH, NPTH, F.Cu at (141.3, 70.1)
- added REF**: NPTH, NPTH, F.Cu at (154.0, 58.1)
- added REF**: NPTH, NPTH, F.Cu at (161.5, 63.2)
- added REF**: NPTH, NPTH, F.Cu at (141.3, 57.4)
- added REF**: NPTH, NPTH, F.Cu at (179.4, 45.4)
- added REF**: NPTH, NPTH, F.Cu at (135.5, 65.0)
- added REF**: NPTH, NPTH, F.Cu at (179.2, 20.6)
- added REF**: NPTH, NPTH, F.Cu at (166.7, 44.7)
- added REF**: NPTH, NPTH, F.Cu at (179.2, 23.3)
- added REF**: NPTH, NPTH, F.Cu at (154.0, 32.0)
- added REF**: NPTH, NPTH, F.Cu at (148.8, 77.7)
- added REF**: NPTH, NPTH, F.Cu at (148.8, 52.3)
- added REF**: NPTH, NPTH, F.Cu at (179.2, 91.1)
- added REF**: NPTH, NPTH, F.Cu at (173.6, 63.2)
- added REF**: NPTH, NPTH, F.Cu at (117.6, 58.1)
- added REF**: NPTH, NPTH, F.Cu at (168.4, 45.4)
- added REF**: NPTH, NPTH, F.Cu at (122.8, 39.6)
- added REF**: NPTH, NPTH, F.Cu at (173.6, 77.7)
- added REF**: NPTH, NPTH, F.Cu at (179.4, 58.1)
- added REF**: NPTH, NPTH, F.Cu at (148.8, 88.6)
- added REF**: Fiducial, Fiducial, F.Cu at (113.3, 93.0)
- added REF**: NPTH, NPTH, F.Cu at (113.5, 88.5)
- added REF**: NPTH, NPTH, F.Cu at (168.4, 32.0)
- added REF**: NPTH, NPTH, F.Cu at (155.7, 44.7)
- added REF**: NPTH, NPTH, F.Cu at (181.8, 88.5)
- added REF**: NPTH, NPTH, F.Cu at (174.2, 75.9)
- added REF**: NPTH, NPTH, F.Cu at (148.2, 52.3)
- added REF**: NPTH, NPTH, F.Cu at (123.4, 37.8)
- added REF**: NPTH, NPTH, F.Cu at (135.5, 63.2)
- added REF**: NPTH, NPTH, F.Cu at (148.2, 50.5)
- added REF**: NPTH, NPTH, F.Cu at (155.7, 45.4)
- added REF**: NPTH, NPTH, F.Cu at (141.3, 32.7)
- added REF**: NPTH, NPTH, F.Cu at (130.3, 57.4)
- added REF**: NPTH, NPTH, F.Cu at (166.7, 58.1)
- added REF**: NPTH, NPTH, F.Cu at (136.1, 88.6)
- added REF**: NPTH, NPTH, F.Cu at (185.1, 27.0)
- added REF**: NPTH, NPTH, F.Cu at (174.2, 77.7)
- added REF**: NPTH, NPTH, F.Cu at (184.6, 27.0)
- added REF**: NPTH, NPTH, F.Cu at (166.7, 45.4)
- added REF**: NPTH, NPTH, F.Cu at (173.6, 39.6)
- added REF**: NPTH, NPTH, F.Cu at (173.6, 52.3)
- added REF**: NPTH, NPTH, F.Cu at (135.5, 39.6)
- added REF**: NPTH, NPTH, F.Cu at (136.1, 63.2)
- added REF**: NPTH, NPTH, F.Cu at (154.0, 57.4)
- added REF**: NPTH, NPTH, F.Cu at (114.1, 88.5)
- added REF**: NPTH, NPTH, F.Cu at (123.4, 50.5)
- added REF**: NPTH, NPTH, F.Cu at (122.8, 52.3)
- added REF**: NPTH, NPTH, F.Cu at (122.8, 65.0)
- added REF**: NPTH, NPTH, F.Cu at (141.3, 82.8)
- added REF**: NPTH, NPTH, F.Cu at (122.8, 37.8)
- added REF**: NPTH, NPTH, F.Cu at (173.6, 65.0)
- added REF**: NPTH, NPTH, F.Cu at (154.0, 70.8)
- added REF**: NPTH, NPTH, F.Cu at (168.4, 70.1)
- added REF**: NPTH, NPTH, F.Cu at (179.2, 94.4)
- added REF**: NPTH, NPTH, F.Cu at (179.4, 32.0)
- added REF**: NPTH, NPTH, F.Cu at (160.9, 26.9)
- added REF**: NPTH, NPTH, F.Cu at (174.2, 50.5)
- added REF**: NPTH, NPTH, F.Cu at (136.1, 39.6)
- added REF**: NPTH, NPTH, F.Cu at (154.0, 82.8)
- added REF**: NPTH, NPTH, F.Cu at (179.2, 93.8)
- added REF**: NPTH, NPTH, F.Cu at (128.6, 32.0)
- added REF**: NPTH, NPTH, F.Cu at (185.7, 27.0)
- added REF**: NPTH, NPTH, F.Cu at (143.0, 45.4)
- added REF**: NPTH, NPTH, F.Cu at (136.1, 26.9)
- added REF**: NPTH, NPTH, F.Cu at (155.7, 70.1)
- added REF**: NPTH, NPTH, F.Cu at (141.3, 32.0)
- added REF**: NPTH, NPTH, F.Cu at (185.1, 88.5)
- added REF**: NPTH, NPTH, F.Cu at (117.8, 23.9)
- added REF**: NPTH, NPTH, F.Cu at (155.7, 70.8)
- added REF**: NPTH, NPTH, F.Cu at (136.1, 77.7)
- added REF**: NPTH, NPTH, F.Cu at (179.4, 70.8)
- added REF**: NPTH, NPTH, F.Cu at (135.5, 50.5)
- added REF**: NPTH, NPTH, F.Cu at (117.8, 94.9)
- added REF**: NPTH, NPTH, F.Cu at (179.2, 21.1)
- added REF**: NPTH, NPTH, F.Cu at (179.2, 22.8)
- added REF**: NPTH, NPTH, F.Cu at (166.7, 82.8)
- added REF**: NPTH, NPTH, F.Cu at (179.2, 92.2)
- added REF**: NPTH, NPTH, F.Cu at (143.0, 44.7)
- added REF**: NPTH, NPTH, F.Cu at (155.7, 32.7)
- added REF**: NPTH, NPTH, F.Cu at (148.8, 65.0)
- added REF**: NPTH, NPTH, F.Cu at (117.6, 45.4)
- added REF**: NPTH, NPTH, F.Cu at (179.2, 91.6)
- added REF**: NPTH, NPTH, F.Cu at (173.6, 37.8)
- added REF**: NPTH, NPTH, F.Cu at (113.0, 88.5)
- added REF**: NPTH, NPTH, F.Cu at (166.7, 32.0)
- added REF**: NPTH, NPTH, F.Cu at (181.8, 27.0)
- added REF**: NPTH, NPTH, F.Cu at (143.0, 32.0)
- added REF**: NPTH, NPTH, F.Cu at (174.2, 52.3)
- added REF**: NPTH, NPTH, F.Cu at (123.4, 63.2)
- added REF**: NPTH, NPTH, F.Cu at (184.0, 27.0)
- added REF**: NPTH, NPTH, F.Cu at (161.5, 52.3)
- added REF**: NPTH, NPTH, F.Cu at (117.6, 82.8)
- added REF**: NPTH, NPTH, F.Cu at (148.8, 37.8)
- added REF**: NPTH, NPTH, F.Cu at (130.3, 45.4)
- added REF**: NPTH, NPTH, F.Cu at (154.0, 45.4)
- added REF**: NPTH, NPTH, F.Cu at (185.7, 88.5)
- added REF**: NPTH, NPTH, F.Cu at (143.0, 58.1)
- added REF**: NPTH, NPTH, F.Cu at (148.8, 75.9)
- added REF**: NPTH, NPTH, F.Cu at (130.3, 32.0)
- added REF**: NPTH, NPTH, F.Cu at (148.8, 50.5)
- added REF**: Fiducial, Fiducial, B.Cu at (113.3, 93.0)
- added REF**: Fiducial, Fiducial, B.Cu at (113.3, 22.5)
- added REF**: Fiducial, Fiducial, B.Cu at (183.7, 22.5)
- added REF**: NPTH, NPTH, F.Cu at (160.9, 88.6)
- added REF**: NPTH, NPTH, F.Cu at (135.5, 26.9)
- added REF**: NPTH, NPTH, F.Cu at (122.8, 63.2)
- added REF**: NPTH, NPTH, F.Cu at (179.2, 93.3)
- added REF**: NPTH, NPTH, F.Cu at (123.4, 75.9)
- added REF**: NPTH, NPTH, F.Cu at (114.6, 27.0)
- added REF**: NPTH, NPTH, F.Cu at (115.2, 27.0)
- added REF**: NPTH, NPTH, F.Cu at (136.1, 75.9)
- added REF**: NPTH, NPTH, F.Cu at (182.4, 27.0)
- added REF**: NPTH, NPTH, F.Cu at (160.9, 37.8)
- added REF**: NPTH, NPTH, F.Cu at (160.9, 63.2)
- added REF**: NPTH, NPTH, F.Cu at (179.2, 21.7)
- added REF**: NPTH, NPTH, F.Cu at (168.4, 32.7)
- added REF**: NPTH, NPTH, F.Cu at (173.6, 75.9)
- added REF**: NPTH, NPTH, F.Cu at (123.4, 52.3)
- added REF**: NPTH, NPTH, F.Cu at (141.3, 83.5)
- added REF**: NPTH, NPTH, F.Cu at (122.8, 88.6)
- added REF**: NPTH, NPTH, F.Cu at (141.3, 70.8)
- added REF**: NPTH, NPTH, F.Cu at (148.2, 77.7)
- added REF**: NPTH, NPTH, F.Cu at (161.5, 75.9)
- added REF**: NPTH, NPTH, F.Cu at (143.0, 70.8)
- added REF**: NPTH, NPTH, F.Cu at (130.3, 70.1)
- added REF**: NPTH, NPTH, F.Cu at (143.0, 57.4)
- added REF**: NPTH, NPTH, F.Cu at (160.9, 77.7)
- added REF**: NPTH, NPTH, F.Cu at (154.0, 70.1)
- added REF**: NPTH, NPTH, F.Cu at (168.4, 44.7)
- added REF**: NPTH, NPTH, F.Cu at (141.3, 44.7)
- added REF**: NPTH, NPTH, F.Cu at (123.4, 39.6)
- added REF**: NPTH, NPTH, F.Cu at (130.3, 44.7)
- added REF**: NPTH, NPTH, F.Cu at (135.5, 77.7)
- added REF**: NPTH, NPTH, F.Cu at (143.0, 82.8)
- added REF**: NPTH, NPTH, F.Cu at (136.1, 50.5)
- added REF**: NPTH, NPTH, F.Cu at (166.7, 32.7)
- added REF**: NPTH, NPTH, F.Cu at (117.6, 32.0)
- added REF**: NPTH, NPTH, F.Cu at (122.8, 77.7)
- added REF**: NPTH, NPTH, F.Cu at (143.0, 70.1)
- added REF**: NPTH, NPTH, F.Cu at (168.4, 58.1)
- added REF**: NPTH, NPTH, F.Cu at (160.9, 75.9)
- added REF**: NPTH, NPTH, F.Cu at (143.0, 83.5)
- added REF**: NPTH, NPTH, F.Cu at (179.4, 57.4)
- added REF**: NPTH, NPTH, F.Cu at (174.2, 26.9)
- added REF**: NPTH, NPTH, F.Cu at (122.8, 50.5)
- added REF**: NPTH, NPTH, F.Cu at (166.7, 70.1)
- added REF**: NPTH, NPTH, F.Cu at (117.6, 70.8)
- added REF**: NPTH, NPTH, F.Cu at (128.6, 70.8)
- added REF**: NPTH, NPTH, F.Cu at (173.6, 26.9)
- added REF**: NPTH, NPTH, F.Cu at (135.5, 37.8)
- added REF**: NPTH, NPTH, F.Cu at (148.8, 63.2)
- added REF**: NPTH, NPTH, F.Cu at (155.7, 57.4)
- added REF**: NPTH, NPTH, F.Cu at (117.6, 32.7)
- added REF**: NPTH, NPTH, F.Cu at (114.6, 88.5)
- added REF**: NPTH, NPTH, F.Cu at (113.0, 27.0)
- added REF**: NPTH, NPTH, F.Cu at (123.4, 77.7)
- added REF**: NPTH, NPTH, F.Cu at (117.8, 20.6)
- added REF**: NPTH, NPTH, F.Cu at (148.2, 75.9)
- added REF**: NPTH, NPTH, F.Cu at (161.5, 39.6)
- added REF**: NPTH, NPTH, F.Cu at (128.6, 82.8)
- added REF**: NPTH, NPTH, F.Cu at (174.2, 88.6)
- added REF**: NPTH, NPTH, F.Cu at (130.3, 32.7)
- added REF**: NPTH, NPTH, F.Cu at (183.5, 88.5)
- added REF**: NPTH, NPTH, F.Cu at (179.4, 32.7)
- added REF**: NPTH, NPTH, F.Cu at (122.8, 26.9)
- added REF**: NPTH, NPTH, F.Cu at (173.6, 50.5)
- added REF**: NPTH, NPTH, F.Cu at (128.6, 44.7)
- added REF**: NPTH, NPTH, F.Cu at (161.5, 50.5)
- added REF**: NPTH, NPTH, F.Cu at (174.2, 37.8)
- added REF**: NPTH, NPTH, F.Cu at (117.8, 24.4)
- added REF**: NPTH, NPTH, F.Cu at (155.7, 82.8)
- added REF**: NPTH, NPTH, F.Cu at (136.1, 37.8)
- added REF**: NPTH, NPTH, F.Cu at (161.5, 77.7)
- added REF**: NPTH, NPTH, F.Cu at (117.8, 91.6)
- added REF**: NPTH, NPTH, F.Cu at (112.4, 27.0)
- added REF**: NPTH, NPTH, F.Cu at (117.8, 92.7)
- added REF**: NPTH, NPTH, F.Cu at (183.5, 27.0)
